Commit message: feat: integrate CAD sorting updates and streamline validation
Align robot geometry, grasp targets, and hand-eye fixtures with the CAD
model. Update sorting, perception, collision handling, and simulation
performance profiles with their implementation documentation.

Consolidate small test suites, remove redundant source assertions, and
keep presentation sources and exports local through Git ignore rules.

Validation: 13 packages built; 912 focused Python checks and 45 CTest
checks passed. Full workspace: 1435 tests, 1 existing wheel speed tracking
failure, 3 skips. Tool checks: 23 passed, 2 skips. Static checks passed.

File: ros2_ws/src/cleany_description/urdf/cleany_geometry.xacro (robot description, xacro)
@@ -1,22 +1,54 @@
-<?xml version="1.0"?>
 <robot xmlns:xacro="http://www.ros.org/wiki/xacro">
-  <xacro:include filename="$(find cleany_description)/urdf/dual_arm.xacro"/>
-  <!-- Backend-neutral physical model shared by all top-level descriptions. -->
-  <xacro:macro name="cleany_robot_geometry" params="">
+  <xacro:include filename="$(find cleany_description)/urdf/physical_properties.xacro" />
+  <xacro:include filename="$(find cleany_description)/urdf/dual_arm.xacro" />
+  <xacro:include filename="$(find cleany_description)/urdf/head_camera.xacro" />
+  <xacro:macro name="cleany_robot_geometry" params="include_wheel_joints:=false">
+    <!-- Fixed mast belongs to every model, including the controller's TF tree. -->
+    <xacro:cleany_head_mount/>
     <link name="base_link">
-      <visual>
-        <origin xyz="0 0 0"/>
-        <geometry><box size="0.6 0.64 0.76"/></geometry>
-        <material name="cleany_white"/>
-      </visual>
-      <collision>
-        <origin xyz="0 0 0"/>
-        <geometry><box size="0.6 0.64 0.76"/></geometry>
-      </collision>
+      <xacro:cleany_link_properties link_name="base_link" />
     </link>
-    <!-- base_link +X is front and physical +Y is left. -->
-    <xacro:cleany_arm side="left" side_sign="1" base_y="0.1552" base_yaw="3.14159265359"/>
-    <!-- base_link +X is front and physical -Y is right. -->
-    <xacro:cleany_arm side="right" side_sign="-1" base_y="-0.1552" base_yaw="0"/>
+    <xacro:cleany_arm side="left" side_sign="1" base_xyz="0.1163 0.185117 0.447797" base_yaw="3.14159265359" />
+    <xacro:cleany_arm side="right" side_sign="-1" base_xyz="0.116101 -0.185063 0.447797" base_yaw="0" />
+    <link name="rear_left_wheel_link">
+      <xacro:cleany_link_properties link_name="rear_left_wheel_link" />
+    </link>
+    <joint name="rear_left_wheel_joint" type="${'continuous' if include_wheel_joints else 'fixed'}">
+      <origin xyz="-0.175025 0.301927 -0.316497" rpy="0 -0 0" />
+      <parent link="base_link" />
+      <child link="rear_left_wheel_link" />
+      <axis xyz="0 1 0" />
+      <limit effort="2.646" velocity="12.017" />
+    </joint>
+    <link name="rear_right_wheel_link">
+      <xacro:cleany_link_properties link_name="rear_right_wheel_link" />
+    </link>
+    <joint name="rear_right_wheel_joint" type="${'continuous' if include_wheel_joints else 'fixed'}">
+      <origin xyz="-0.175025 -0.301873 -0.316497" rpy="0 -0 0" />
+      <parent link="base_link" />
+      <child link="rear_right_wheel_link" />
+      <axis xyz="0 1 0" />
+      <limit effort="2.646" velocity="12.017" />
+    </joint>
+    <link name="front_left_wheel_link">
+      <xacro:cleany_link_properties link_name="front_left_wheel_link" />
+    </link>
+    <joint name="front_left_wheel_joint" type="${'continuous' if include_wheel_joints else 'fixed'}">
+      <origin xyz="0.174975 0.301927 -0.316497" rpy="0 -0 0" />
+      <parent link="base_link" />
+      <child link="front_left_wheel_link" />
+      <axis xyz="0 1 0" />
+      <limit effort="2.646" velocity="12.017" />
+    </joint>
+    <link name="front_right_wheel_link">
+      <xacro:cleany_link_properties link_name="front_right_wheel_link" />
+    </link>
+    <joint name="front_right_wheel_joint" type="${'continuous' if include_wheel_joints else 'fixed'}">
+      <origin xyz="0.174975 -0.301873 -0.316497" rpy="0 -0 0" />
+      <parent link="base_link" />
+      <child link="front_right_wheel_link" />
+      <axis xyz="0 1 0" />
+      <limit effort="2.646" velocity="12.017" />
+    </joint>
   </xacro:macro>
 </robot>

File: ros2_ws/src/cleany_description/urdf/dual_arm.xacro (robot description, xacro)
@@ -1,209 +1,82 @@
-<?xml version="1.0"?>
 <robot xmlns:xacro="http://www.ros.org/wiki/xacro">
-  <!--
-    The origin/axis values below are the canonical ROS representation of the
-    MuJoCo body-local joints in mjcf/cleany.xml.  side_sign is +1 on physical
-    +Y (left) and -1 on physical -Y (right).
-  -->
-  <!-- Motors are separate CAD parts. Include them in the collision model so
-       RGB-D robot self-filtering does not insert their surfaces into OctoMap. -->
-  <xacro:macro name="cleany_arm_motor" params="mesh xyz:='0 0 0'">
-    <visual>
-      <origin xyz="${xyz}"/>
-      <geometry><mesh filename="package://cleany_description/meshes/${mesh}.stl"/></geometry>
-      <material name="cleany_motor"/>
-    </visual>
-    <collision>
-      <origin xyz="${xyz}"/>
-      <geometry><mesh filename="package://cleany_description/meshes/${mesh}.stl"/></geometry>
-    </collision>
-  </xacro:macro>
-  <!-- Camera meshes are rigidly mounted on the gripper. Compose the MJCF
-       camera-body and geom origins here without adding control joints. -->
-  <xacro:macro name="cleany_wrist_camera_mesh" params="mesh material side">
-    <visual>
-      <origin xyz="0 ${-0.007 if side == 'left' else -0.006} 0.024"
-              rpy="1.57079632679 0 -1.57079632679"/>
-      <geometry><mesh filename="package://cleany_description/meshes/${mesh}.stl" scale="0.001 0.001 0.001"/></geometry>
-      <material name="${material}"/>
-    </visual>
-    <collision>
-      <origin xyz="0 ${-0.007 if side == 'left' else -0.006} 0.024"
-              rpy="1.57079632679 0 -1.57079632679"/>
-      <geometry><mesh filename="package://cleany_description/meshes/${mesh}.stl" scale="0.001 0.001 0.001"/></geometry>
-    </collision>
-  </xacro:macro>
-  <xacro:macro name="cleany_arm" params="side side_sign base_y base_yaw">
+  <xacro:macro name="cleany_arm" params="side side_sign base_xyz base_yaw">
     <link name="${side}_shoulder_yaw_link">
-      <inertial>
-        <origin xyz="0 0 0"/>
-        <mass value="0.099"/>
-        <inertia ixx="0.0001" ixy="0" ixz="0" iyy="0.0001" iyz="0" izz="0.0001"/>
-      </inertial>
-      <visual>
-        <geometry><mesh filename="package://cleany_description/meshes/Rotation_Pitch.stl"/></geometry>
-        <material name="cleany_white"/>
-      </visual>
-      <collision>
-        <geometry><mesh filename="package://cleany_description/meshes/Rotation_Pitch.stl.convex.stl"/></geometry>
-      </collision>
-      <xacro:cleany_arm_motor mesh="Rotation_Pitch_Motor"/>
+      <xacro:cleany_link_properties link_name="${side}_shoulder_yaw_link" />
     </link>
     <joint name="${side}_shoulder_yaw_joint" type="revolute">
-      <parent link="base_link"/>
-      <child link="${side}_shoulder_yaw_link"/>
-      <origin xyz="0.09 ${base_y} 0.4115" rpy="1.57079632679 0 ${base_yaw}"/>
-      <!-- Positive shoulder yaw is counter-clockwise about base_link +Z. -->
-      <axis xyz="0 1 0"/>
-      <limit lower="-2.16" upper="2.16" effort="2.6477955" velocity="4.245"/>
+      <parent link="base_link" />
+      <child link="${side}_shoulder_yaw_link" />
+      <origin xyz="${base_xyz}" rpy="1.57079632679 0 ${base_yaw}" />
+      <axis xyz="0 1 0" />
+      <limit lower="-2.16" upper="2.16" effort="2.6477955" velocity="4.245" />
     </joint>
     <link name="${side}_upper_arm_link">
-      <inertial>
-        <origin xyz="0.00011909447145 0.13366336448 0.00941424883693"/>
-        <mass value="0.1185"/>
-        <inertia ixx="0.000344882383932" ixy="0.0000000126253142805" ixz="-0.0000000018457009038"
-                 iyy="0.0000390640385918" iyz="-0.0000322497618493" izz="0.000341356582549"/>
-      </inertial>
-      <visual>
-        <origin xyz="-0.0001 0.0651 -0.012" rpy="1.57079632679 0 -1.57079632679"/>
-        <geometry><mesh filename="package://cleany_description/meshes/Upper_Arm_5cm_Sockets.stl"/></geometry>
-        <material name="cleany_white"/>
-      </visual>
-      <visual>
-        <origin xyz="-0.0001 0.0651 -0.012" rpy="1.57079632679 0 -1.57079632679"/>
-        <geometry><mesh filename="package://cleany_description/meshes/Upper_Arm_5cm_Carbon.stl"/></geometry>
-        <material name="cleany_carbon"/>
-      </visual>
-      <collision>
-        <origin xyz="-0.0001 0.0651 -0.012" rpy="1.57079632679 0 -1.57079632679"/>
-        <geometry><mesh filename="package://cleany_description/meshes/Upper_Arm_5cm.stl"/></geometry>
-      </collision>
-      <xacro:cleany_arm_motor mesh="Upper_Arm_Motor" xyz="0 0.05 0"/>
+      <xacro:cleany_link_properties link_name="${side}_upper_arm_link" />
     </link>
     <joint name="${side}_shoulder_pitch_joint" type="revolute">
-      <parent link="${side}_shoulder_yaw_link"/>
-      <child link="${side}_upper_arm_link"/>
-      <origin xyz="0 0.1025 0.0306" rpy="1.57079632679 0 0"/>
-      <axis xyz="-1 0 0"/>
-      <limit lower="-0.22" upper="3.37" effort="4.4129925" velocity="7.086"/>
+      <parent link="${side}_shoulder_yaw_link" />
+      <child link="${side}_upper_arm_link" />
+      <origin xyz="0 0.1025 0.0306" rpy="1.57079632679 0 0" />
+      <axis xyz="-1 0 0" />
+      <limit lower="-0.22" upper="3.37" effort="4.4129925" velocity="7.086" />
     </joint>
     <link name="${side}_lower_arm_link">
-      <inertial>
-        <origin xyz="-0.000705377693495 0.003222361186 0.133834080359"/>
-        <mass value="0.093"/>
-        <inertia ixx="0.000317919847018" ixy="-0.000000245304506082" ixz="-0.00000442747241607"
-                 iyy="0.000326130407587" iyz="-0.000011286233547" izz="0.0000182344857592"/>
-      </inertial>
-      <visual>
-        <origin xyz="-0.0025 0.032 0.065" rpy="0 1.57079632679 0"/>
-        <geometry><mesh filename="package://cleany_description/meshes/Lower_Arm_5cm_Sockets.stl"/></geometry>
-        <material name="cleany_white"/>
-      </visual>
-      <visual>
-        <origin xyz="-0.0025 0.032 0.065" rpy="0 1.57079632679 0"/>
-        <geometry><mesh filename="package://cleany_description/meshes/Lower_Arm_5cm_Carbon.stl"/></geometry>
-        <material name="cleany_carbon"/>
-      </visual>
-      <collision>
-        <origin xyz="-0.0025 0.032 0.065" rpy="0 1.57079632679 0"/>
-        <geometry><mesh filename="package://cleany_description/meshes/Lower_Arm_5cm.stl"/></geometry>
-      </collision>
-      <xacro:cleany_arm_motor mesh="Lower_Arm_Motor" xyz="0 0 0.05"/>
+      <xacro:cleany_link_properties link_name="${side}_lower_arm_link" />
     </link>
     <joint name="${side}_elbow_pitch_joint" type="revolute">
-      <parent link="${side}_upper_arm_link"/>
-      <child link="${side}_lower_arm_link"/>
-      <origin xyz="0 0.16257 0.028" rpy="-1.57079632679 0 0"/>
-      <axis xyz="1 0 0"/>
-      <limit lower="-0.22" upper="3.14" effort="4.4129925" velocity="7.086"/>
+      <parent link="${side}_upper_arm_link" />
+      <child link="${side}_lower_arm_link" />
+      <origin xyz="0 0.16257 0.028" rpy="-1.57079632679 0 0" />
+      <axis xyz="1 0 0" />
+      <limit lower="-0.22" upper="3.14" effort="4.4129925" velocity="7.086" />
     </joint>
     <link name="${side}_wrist_pitch_link">
-      <inertial>
-        <origin xyz="-0.000103312 -0.0386143 0.0281156"/>
-        <mass value="0.079"/>
-        <inertia ixx="0.0000368263" ixy="0.000000017893" ixz="-0.0000000528128"
-                 iyy="0.000025391" iyz="0.0000036412" izz="0.000021"/>
-      </inertial>
-      <visual>
-        <geometry><mesh filename="package://cleany_description/meshes/Wrist_Pitch_Roll.stl"/></geometry>
-        <material name="cleany_white"/>
-      </visual>
-      <collision>
-        <geometry><mesh filename="package://cleany_description/meshes/Wrist_Pitch_Roll.stl.convex.stl"/></geometry>
-      </collision>
-      <xacro:cleany_arm_motor mesh="Wrist_Pitch_Roll_Motor"/>
+      <xacro:cleany_link_properties link_name="${side}_wrist_pitch_link" />
     </link>
     <joint name="${side}_wrist_pitch_joint" type="revolute">
-      <parent link="${side}_lower_arm_link"/>
-      <child link="${side}_wrist_pitch_link"/>
-      <origin xyz="0 0.0052 0.1849" rpy="-1.57079632679 0 0"/>
-      <axis xyz="1 0 0"/>
-      <limit lower="-1.65806284946" upper="1.65806272933" effort="2.6477955" velocity="4.245"/>
+      <parent link="${side}_lower_arm_link" />
+      <child link="${side}_wrist_pitch_link" />
+      <origin xyz="0 0.0052 0.1849" rpy="-1.57079632679 0 0" />
+      <axis xyz="1 0 0" />
+      <limit lower="-1.65806284946" upper="1.65806272933" effort="2.6477955" velocity="4.245" />
     </joint>
     <link name="${side}_gripper_frame">
-      <inertial>
-        <origin xyz="0 0 0"/>
-        <mass value="0.06"/>
-        <inertia ixx="0.00004" ixy="0" ixz="0" iyy="0.00004" iyz="0" izz="0.00004"/>
-      </inertial>
-      <visual>
-        <geometry><mesh filename="package://cleany_description/meshes/Fixed_Jaw.stl"/></geometry>
-        <material name="cleany_white"/>
-      </visual>
-      <collision>
-        <geometry><mesh filename="package://cleany_description/meshes/Fixed_Jaw.stl.convex.stl"/></geometry>
-      </collision>
-      <xacro:cleany_arm_motor mesh="Fixed_Jaw_Motor"/>
-      <xacro:cleany_wrist_camera_mesh mesh="XLeRobot_camera1" material="cleany_white" side="${side}"/>
-      <xacro:cleany_wrist_camera_mesh mesh="XLeRobot_camera2" material="cleany_motor" side="${side}"/>
+      <xacro:cleany_link_properties link_name="${side}_gripper_frame" />
     </link>
     <joint name="${side}_wrist_roll_joint" type="revolute">
-      <parent link="${side}_wrist_pitch_link"/>
-      <child link="${side}_gripper_frame"/>
-      <origin xyz="0 -0.0601 0" rpy="0 1.57079632679 0"/>
-      <axis xyz="0 -1 0"/>
-      <limit lower="-2.743847297" upper="2.84120630938" effort="2.6477955" velocity="4.245"/>
+      <parent link="${side}_wrist_pitch_link" />
+      <child link="${side}_gripper_frame" />
+      <origin xyz="0 -0.0601 0" rpy="0 1.57079632679 0" />
+      <axis xyz="0 -1 0" />
+      <limit lower="-2.743847297" upper="2.84120630938" effort="2.6477955" velocity="4.245" />
     </joint>
     <link name="${side}_moving_jaw_link">
-      <inertial>
-        <origin xyz="0 0 0"/>
-        <mass value="0.02"/>
-        <inertia ixx="0.00001" ixy="0" ixz="0" iyy="0.00001" iyz="0" izz="0.00001"/>
-      </inertial>
-      <visual>
-        <geometry><mesh filename="package://cleany_description/meshes/Moving_Jaw.stl"/></geometry>
-        <material name="cleany_white"/>
-      </visual>
-      <collision>
-        <geometry><mesh filename="package://cleany_description/meshes/Moving_Jaw.stl.convex.stl"/></geometry>
-      </collision>
+      <xacro:cleany_link_properties link_name="${side}_moving_jaw_link" />
     </link>
     <joint name="${side}_gripper_joint" type="revolute">
-      <parent link="${side}_gripper_frame"/>
-      <child link="${side}_moving_jaw_link"/>
-      <!-- Convert MJCF intrinsic xyz Rx(3.1416)*Rz(3.33) to URDF
-           fixed-axis Rz*Ry*Rx, preserving the rounded CAD roll exactly. -->
-      <origin xyz="-0.0202 -0.0244 0" rpy="3.141585437183305 -0.000001375943427901895 2.953185307184551"/>
-      <axis xyz="0 0 1"/>
-      <limit lower="-0.374532977628" upper="1.74532919957" effort="2.6477955" velocity="4.245"/>
+      <parent link="${side}_gripper_frame" />
+      <child link="${side}_moving_jaw_link" />
+      <origin xyz="-0.0202 -0.0244 0" rpy="3.14159265359 0 3.33" />
+      <axis xyz="0 0 1" />
+      <limit lower="-0.374532977628" upper="1.74532919957" effort="2.6477955" velocity="4.245" />
     </joint>
-    <!-- Nominal midpoint between the jaw tips; not a hardware calibration. -->
-    <link name="${side}_grasp_tcp"/>
+    <link name="${side}_grasp_tcp">
+      <xacro:cleany_link_properties link_name="${side}_grasp_tcp" />
+    </link>
     <joint name="${side}_grasp_tcp_joint" type="fixed">
-      <parent link="${side}_gripper_frame"/>
-      <child link="${side}_grasp_tcp"/>
-      <origin xyz="0 -0.100 0" rpy="0 0 0"/>
+      <parent link="${side}_gripper_frame" />
+      <child link="${side}_grasp_tcp" />
+      <origin xyz="0 -0.100 0" rpy="0 0 0" />
     </joint>
-    <!--
-      Position-only IK cannot constrain a 5-DOF arm's complete quaternion.
-      Placing this collision-free virtual tip on the grasp point makes the
-      physical TCP stand 140 mm back while its -Y approach axis points at it.
-    -->
-    <link name="${side}_pregrasp_aim_tip"/>
+    <link name="${side}_pregrasp_aim_tip">
+      <xacro:cleany_link_properties link_name="${side}_pregrasp_aim_tip" />
+    </link>
     <joint name="${side}_pregrasp_aim_tip_joint" type="fixed">
-      <parent link="${side}_grasp_tcp"/>
-      <child link="${side}_pregrasp_aim_tip"/>
-      <origin xyz="0 -0.140 0" rpy="0 0 0"/>
+      <parent link="${side}_grasp_tcp" />
+      <child link="${side}_pregrasp_aim_tip" />
+      <origin xyz="0 -0.140 0" rpy="0 0 0" />
     </joint>
+    <!-- Wrist camera extrinsics are evaluation-only until calibrated.
+         Do not publish the MJCF ground-truth optical edge into runtime TF. -->
   </xacro:macro>
 </robot>
