Commit message: feat(grasp): stabilize AnyGrasp-ready 6-DoF pregrasp execution

File: ros2_ws/src/cleany_description/urdf/cleany_control.urdf.xacro (robot description, xacro)
@@ -8,4 +8,16 @@
   <xacro:arg name="camera_frame_name" default="left_wrist_rgb_vendor_frame"/>
   <xacro:arg name="enable_gripper_command" default="false"/>
+  <xacro:arg name="left_shoulder_yaw_initial" default="0.0"/>
+  <xacro:arg name="left_shoulder_pitch_initial" default="0.0"/>
+  <xacro:arg name="left_elbow_pitch_initial" default="0.0"/>
+  <xacro:arg name="left_wrist_pitch_initial" default="0.0"/>
+  <xacro:arg name="left_wrist_roll_initial" default="0.0"/>
+  <xacro:arg name="left_gripper_initial" default="0.0"/>
+  <xacro:arg name="right_shoulder_yaw_initial" default="0.0"/>
+  <xacro:arg name="right_shoulder_pitch_initial" default="0.0"/>
+  <xacro:arg name="right_elbow_pitch_initial" default="0.0"/>
+  <xacro:arg name="right_wrist_pitch_initial" default="0.0"/>
+  <xacro:arg name="right_wrist_roll_initial" default="0.0"/>
+  <xacro:arg name="right_gripper_initial" default="0.0"/>
   <xacro:include filename="$(find cleany_description)/urdf/materials.xacro"/>
   <xacro:include filename="$(find cleany_description)/urdf/cleany_geometry.xacro"/>
@@ -19,4 +31,16 @@
     camera_name="$(arg camera_name)"
     camera_frame_name="$(arg camera_frame_name)"
-    enable_gripper_command="$(arg enable_gripper_command)"/>
+    enable_gripper_command="$(arg enable_gripper_command)"
+    left_shoulder_yaw_initial="$(arg left_shoulder_yaw_initial)"
+    left_shoulder_pitch_initial="$(arg left_shoulder_pitch_initial)"
+    left_elbow_pitch_initial="$(arg left_elbow_pitch_initial)"
+    left_wrist_pitch_initial="$(arg left_wrist_pitch_initial)"
+    left_wrist_roll_initial="$(arg left_wrist_roll_initial)"
+    left_gripper_initial="$(arg left_gripper_initial)"
+    right_shoulder_yaw_initial="$(arg right_shoulder_yaw_initial)"
+    right_shoulder_pitch_initial="$(arg right_shoulder_pitch_initial)"
+    right_elbow_pitch_initial="$(arg right_elbow_pitch_initial)"
+    right_wrist_pitch_initial="$(arg right_wrist_pitch_initial)"
+    right_wrist_roll_initial="$(arg right_wrist_roll_initial)"
+    right_gripper_initial="$(arg right_gripper_initial)"/>
 </robot>

File: ros2_ws/src/cleany_description/urdf/cleany_mujoco_ros2_control.xacro (robot description, xacro)
@@ -1,17 +1,17 @@
 <?xml version="1.0"?>
 <robot xmlns:xacro="http://www.ros.org/wiki/xacro">
-  <xacro:macro name="cleany_mujoco_arm_joint" params="joint_name">
+  <xacro:macro name="cleany_mujoco_arm_joint" params="joint_name initial_value">
     <joint name="${joint_name}">
       <command_interface name="position"/>
       <state_interface name="position">
-        <param name="initial_value">0.0</param>
+        <param name="initial_value">${initial_value}</param>
       </state_interface>
       <state_interface name="velocity"/>
     </joint>
   </xacro:macro>
-  <xacro:macro name="cleany_mujoco_read_only_joint" params="joint_name">
+  <xacro:macro name="cleany_mujoco_read_only_joint" params="joint_name initial_value">
     <joint name="${joint_name}">
       <state_interface name="position">
-        <param name="initial_value">0.0</param>
+        <param name="initial_value">${initial_value}</param>
       </state_interface>
       <state_interface name="velocity"/>
@@ -20,5 +20,7 @@
   <xacro:macro
     name="cleany_mujoco_ros2_control"
-    params="mujoco_model headless sim_speed_factor camera_publish_rate camera_name camera_frame_name enable_gripper_command">
+    params="mujoco_model headless sim_speed_factor camera_publish_rate camera_name camera_frame_name enable_gripper_command
+            left_shoulder_yaw_initial left_shoulder_pitch_initial left_elbow_pitch_initial left_wrist_pitch_initial left_wrist_roll_initial left_gripper_initial
+            right_shoulder_yaw_initial right_shoulder_pitch_initial right_elbow_pitch_initial right_wrist_pitch_initial right_wrist_roll_initial right_gripper_initial">
     <ros2_control name="MujocoSystem" type="system">
       <hardware>
@@ -38,21 +40,21 @@
         <param name="depth_topic">/${camera_name}/depth</param>
       </sensor>
-      <xacro:cleany_mujoco_arm_joint joint_name="left_shoulder_yaw_joint"/>
-      <xacro:cleany_mujoco_arm_joint joint_name="left_shoulder_pitch_joint"/>
-      <xacro:cleany_mujoco_arm_joint joint_name="left_elbow_pitch_joint"/>
-      <xacro:cleany_mujoco_arm_joint joint_name="left_wrist_pitch_joint"/>
-      <xacro:cleany_mujoco_arm_joint joint_name="left_wrist_roll_joint"/>
-      <xacro:cleany_mujoco_arm_joint joint_name="right_shoulder_yaw_joint"/>
-      <xacro:cleany_mujoco_arm_joint joint_name="right_shoulder_pitch_joint"/>
-      <xacro:cleany_mujoco_arm_joint joint_name="right_elbow_pitch_joint"/>
-      <xacro:cleany_mujoco_arm_joint joint_name="right_wrist_pitch_joint"/>
-      <xacro:cleany_mujoco_arm_joint joint_name="right_wrist_roll_joint"/>
+      <xacro:cleany_mujoco_arm_joint joint_name="left_shoulder_yaw_joint" initial_value="${left_shoulder_yaw_initial}"/>
+      <xacro:cleany_mujoco_arm_joint joint_name="left_shoulder_pitch_joint" initial_value="${left_shoulder_pitch_initial}"/>
+      <xacro:cleany_mujoco_arm_joint joint_name="left_elbow_pitch_joint" initial_value="${left_elbow_pitch_initial}"/>
+      <xacro:cleany_mujoco_arm_joint joint_name="left_wrist_pitch_joint" initial_value="${left_wrist_pitch_initial}"/>
+      <xacro:cleany_mujoco_arm_joint joint_name="left_wrist_roll_joint" initial_value="${left_wrist_roll_initial}"/>
+      <xacro:cleany_mujoco_arm_joint joint_name="right_shoulder_yaw_joint" initial_value="${right_shoulder_yaw_initial}"/>
+      <xacro:cleany_mujoco_arm_joint joint_name="right_shoulder_pitch_joint" initial_value="${right_shoulder_pitch_initial}"/>
+      <xacro:cleany_mujoco_arm_joint joint_name="right_elbow_pitch_joint" initial_value="${right_elbow_pitch_initial}"/>
+      <xacro:cleany_mujoco_arm_joint joint_name="right_wrist_pitch_joint" initial_value="${right_wrist_pitch_initial}"/>
+      <xacro:cleany_mujoco_arm_joint joint_name="right_wrist_roll_joint" initial_value="${right_wrist_roll_initial}"/>
       <xacro:if value="${enable_gripper_command}">
-        <xacro:cleany_mujoco_arm_joint joint_name="left_gripper_joint"/>
-        <xacro:cleany_mujoco_arm_joint joint_name="right_gripper_joint"/>
+        <xacro:cleany_mujoco_arm_joint joint_name="left_gripper_joint" initial_value="${left_gripper_initial}"/>
+        <xacro:cleany_mujoco_arm_joint joint_name="right_gripper_joint" initial_value="${right_gripper_initial}"/>
       </xacro:if>
       <xacro:unless value="${enable_gripper_command}">
-        <xacro:cleany_mujoco_read_only_joint joint_name="left_gripper_joint"/>
-        <xacro:cleany_mujoco_read_only_joint joint_name="right_gripper_joint"/>
+        <xacro:cleany_mujoco_read_only_joint joint_name="left_gripper_joint" initial_value="${left_gripper_initial}"/>
+        <xacro:cleany_mujoco_read_only_joint joint_name="right_gripper_joint" initial_value="${right_gripper_initial}"/>
       </xacro:unless>
     </ros2_control>

Commit message: feat: integrate sensor-based sorting and Jetson perception profiles
Add observed geometry, wrist tracking, collision mapping, and rear collection shelf fixtures. Unify Gemini Flash-Lite and SAM2-tiny configuration, support external GPU perception, and refresh runtime documentation.

Validation: 766 Python and 44 C++ focused tests passed; container contract checks passed with two Compose checks skipped. Jetson hardware and end-to-end rear collection remain unverified.

File: ros2_ws/src/cleany_description/urdf/cleany_control.urdf.xacro (robot description, xacro)
@@ -2,7 +2,9 @@
 <robot name="cleany" xmlns:xacro="http://www.ros.org/wiki/xacro">
   <xacro:arg name="mujoco_model" default=""/>
+  <xacro:arg name="mujoco_hardware_plugin" default="mujoco_ros2_control/MujocoSystemInterface"/>
   <xacro:arg name="headless" default="true"/>
   <xacro:arg name="sim_speed_factor" default="1.0"/>
   <xacro:arg name="camera_publish_rate" default="10.0"/>
+  <xacro:arg name="scheduled_cameras" default="false"/>
   <xacro:arg name="camera_name" default="left_wrist_rgb"/>
   <xacro:arg name="camera_frame_name" default="left_wrist_rgb_vendor_frame"/>
@@ -26,7 +28,9 @@
   <xacro:cleany_mujoco_ros2_control
     mujoco_model="$(arg mujoco_model)"
+    hardware_plugin="$(arg mujoco_hardware_plugin)"
     headless="$(arg headless)"
     sim_speed_factor="$(arg sim_speed_factor)"
     camera_publish_rate="$(arg camera_publish_rate)"
+    scheduled_cameras="$(arg scheduled_cameras)"
     camera_name="$(arg camera_name)"
     camera_frame_name="$(arg camera_frame_name)"

File: ros2_ws/src/cleany_description/urdf/cleany_mujoco_ros2_control.xacro (robot description, xacro)
@@ -22,12 +22,16 @@
     params="mujoco_model headless sim_speed_factor camera_publish_rate camera_name camera_frame_name enable_gripper_command
             left_shoulder_yaw_initial left_shoulder_pitch_initial left_elbow_pitch_initial left_wrist_pitch_initial left_wrist_roll_initial left_gripper_initial
-            right_shoulder_yaw_initial right_shoulder_pitch_initial right_elbow_pitch_initial right_wrist_pitch_initial right_wrist_roll_initial right_gripper_initial">
+            right_shoulder_yaw_initial right_shoulder_pitch_initial right_elbow_pitch_initial right_wrist_pitch_initial right_wrist_roll_initial right_gripper_initial
+            hardware_plugin:=mujoco_ros2_control/MujocoSystemInterface scheduled_cameras:=false">
     <ros2_control name="MujocoSystem" type="system">
       <hardware>
-        <plugin>mujoco_ros2_control/MujocoSystemInterface</plugin>
+        <plugin>${hardware_plugin}</plugin>
         <param name="mujoco_model">${mujoco_model}</param>
         <param name="headless">${headless}</param>
         <param name="sim_speed_factor">${sim_speed_factor}</param>
         <param name="camera_publish_rate">${camera_publish_rate}</param>
+        <xacro:if value="${scheduled_cameras}">
+          <param name="scheduled_cameras">true</param>
+        </xacro:if>
         <param name="initial_keyframe">handeye_ros2_control_home</param>
       </hardware>

File: ros2_ws/src/cleany_description/urdf/dual_arm.xacro (robot description, xacro)
@@ -6,4 +6,32 @@
     +Y (left) and -1 on physical -Y (right).
   -->
+  <!-- Motors are separate CAD parts. Include them in the collision model so
+       RGB-D robot self-filtering does not insert their surfaces into OctoMap. -->
+  <xacro:macro name="cleany_arm_motor" params="mesh xyz:='0 0 0'">
+    <visual>
+      <origin xyz="${xyz}"/>
+      <geometry><mesh filename="package://cleany_description/meshes/${mesh}.stl"/></geometry>
+      <material name="cleany_motor"/>
+    </visual>
+    <collision>
+      <origin xyz="${xyz}"/>
+      <geometry><mesh filename="package://cleany_description/meshes/${mesh}.stl"/></geometry>
+    </collision>
+  </xacro:macro>
+  <!-- Camera meshes are rigidly mounted on the gripper. Compose the MJCF
+       camera-body and geom origins here without adding control joints. -->
+  <xacro:macro name="cleany_wrist_camera_mesh" params="mesh material side">
+    <visual>
+      <origin xyz="0 ${-0.007 if side == 'left' else -0.006} 0.024"
+              rpy="1.57079632679 0 -1.57079632679"/>
+      <geometry><mesh filename="package://cleany_description/meshes/${mesh}.stl" scale="0.001 0.001 0.001"/></geometry>
+      <material name="${material}"/>
+    </visual>
+    <collision>
+      <origin xyz="0 ${-0.007 if side == 'left' else -0.006} 0.024"
+              rpy="1.57079632679 0 -1.57079632679"/>
+      <geometry><mesh filename="package://cleany_description/meshes/${mesh}.stl" scale="0.001 0.001 0.001"/></geometry>
+    </collision>
+  </xacro:macro>
   <xacro:macro name="cleany_arm" params="side side_sign base_y base_yaw">
     <link name="${side}_shoulder_yaw_link">
@@ -20,4 +48,5 @@
         <geometry><mesh filename="package://cleany_description/meshes/Rotation_Pitch.stl.convex.stl"/></geometry>
       </collision>
+      <xacro:cleany_arm_motor mesh="Rotation_Pitch_Motor"/>
     </link>
     <joint name="${side}_shoulder_yaw_joint" type="revolute">
@@ -50,4 +79,5 @@
         <geometry><mesh filename="package://cleany_description/meshes/Upper_Arm_5cm.stl"/></geometry>
       </collision>
+      <xacro:cleany_arm_motor mesh="Upper_Arm_Motor" xyz="0 0.05 0"/>
     </link>
     <joint name="${side}_shoulder_pitch_joint" type="revolute">
@@ -79,4 +109,5 @@
         <geometry><mesh filename="package://cleany_description/meshes/Lower_Arm_5cm.stl"/></geometry>
       </collision>
+      <xacro:cleany_arm_motor mesh="Lower_Arm_Motor" xyz="0 0 0.05"/>
     </link>
     <joint name="${side}_elbow_pitch_joint" type="revolute">
@@ -101,4 +132,5 @@
         <geometry><mesh filename="package://cleany_description/meshes/Wrist_Pitch_Roll.stl.convex.stl"/></geometry>
       </collision>
+      <xacro:cleany_arm_motor mesh="Wrist_Pitch_Roll_Motor"/>
     </link>
     <joint name="${side}_wrist_pitch_joint" type="revolute">
@@ -122,4 +154,7 @@
         <geometry><mesh filename="package://cleany_description/meshes/Fixed_Jaw.stl.convex.stl"/></geometry>
       </collision>
+      <xacro:cleany_arm_motor mesh="Fixed_Jaw_Motor"/>
+      <xacro:cleany_wrist_camera_mesh mesh="XLeRobot_camera1" material="cleany_white" side="${side}"/>
+      <xacro:cleany_wrist_camera_mesh mesh="XLeRobot_camera2" material="cleany_motor" side="${side}"/>
     </link>
     <joint name="${side}_wrist_roll_joint" type="revolute">
@@ -147,5 +182,7 @@
       <parent link="${side}_gripper_frame"/>
       <child link="${side}_moving_jaw_link"/>
-      <origin xyz="-0.0202 -0.0244 0" rpy="3.14159265359 0 3.33"/>
+      <!-- Convert MJCF intrinsic xyz Rx(3.1416)*Rz(3.33) to URDF
+           fixed-axis Rz*Ry*Rx, preserving the rounded CAD roll exactly. -->
+      <origin xyz="-0.0202 -0.0244 0" rpy="3.141585437183305 -0.000001375943427901895 2.953185307184551"/>
       <axis xyz="0 0 1"/>
       <limit lower="-0.374532977628" upper="1.74532919957" effort="2.6477955" velocity="4.245"/>
