Commit message: feat(sim): integrate MuJoCo study-cafe perception and sorting
Consolidate the validated simulation changes on main while preserving the resolved model, perception and navigation integration. Exclude KB and the manipulation Action server implementation.

File: ros2_ws/src/cleany_description/urdf/cleany_control.urdf.xacro (robot description, xacro)
@@ -2,10 +2,24 @@
 <robot name="cleany" xmlns:xacro="http://www.ros.org/wiki/xacro">
   <xacro:arg name="mujoco_model" default=""/>
+  <xacro:arg name="mujoco_hardware_plugin" default="mujoco_ros2_control/MujocoSystemInterface"/>
   <xacro:arg name="headless" default="true"/>
   <xacro:arg name="sim_speed_factor" default="1.0"/>
   <xacro:arg name="camera_publish_rate" default="10.0"/>
+  <xacro:arg name="scheduled_cameras" default="false"/>
   <xacro:arg name="camera_name" default="left_wrist_rgb"/>
   <xacro:arg name="camera_frame_name" default="left_wrist_rgb_vendor_frame"/>
   <xacro:arg name="enable_gripper_command" default="false"/>
+  <xacro:arg name="left_shoulder_yaw_initial" default="0.0"/>
+  <xacro:arg name="left_shoulder_pitch_initial" default="0.0"/>
+  <xacro:arg name="left_elbow_pitch_initial" default="0.0"/>
+  <xacro:arg name="left_wrist_pitch_initial" default="0.0"/>
+  <xacro:arg name="left_wrist_roll_initial" default="0.0"/>
+  <xacro:arg name="left_gripper_initial" default="0.0"/>
+  <xacro:arg name="right_shoulder_yaw_initial" default="0.0"/>
+  <xacro:arg name="right_shoulder_pitch_initial" default="0.0"/>
+  <xacro:arg name="right_elbow_pitch_initial" default="0.0"/>
+  <xacro:arg name="right_wrist_pitch_initial" default="0.0"/>
+  <xacro:arg name="right_wrist_roll_initial" default="0.0"/>
+  <xacro:arg name="right_gripper_initial" default="0.0"/>
   <xacro:include filename="$(find cleany_description)/urdf/materials.xacro"/>
   <xacro:include filename="$(find cleany_description)/urdf/cleany_geometry.xacro"/>
@@ -14,9 +28,23 @@
   <xacro:cleany_mujoco_ros2_control
     mujoco_model="$(arg mujoco_model)"
+    hardware_plugin="$(arg mujoco_hardware_plugin)"
     headless="$(arg headless)"
     sim_speed_factor="$(arg sim_speed_factor)"
     camera_publish_rate="$(arg camera_publish_rate)"
+    scheduled_cameras="$(arg scheduled_cameras)"
     camera_name="$(arg camera_name)"
     camera_frame_name="$(arg camera_frame_name)"
-    enable_gripper_command="$(arg enable_gripper_command)"/>
+    enable_gripper_command="$(arg enable_gripper_command)"
+    left_shoulder_yaw_initial="$(arg left_shoulder_yaw_initial)"
+    left_shoulder_pitch_initial="$(arg left_shoulder_pitch_initial)"
+    left_elbow_pitch_initial="$(arg left_elbow_pitch_initial)"
+    left_wrist_pitch_initial="$(arg left_wrist_pitch_initial)"
+    left_wrist_roll_initial="$(arg left_wrist_roll_initial)"
+    left_gripper_initial="$(arg left_gripper_initial)"
+    right_shoulder_yaw_initial="$(arg right_shoulder_yaw_initial)"
+    right_shoulder_pitch_initial="$(arg right_shoulder_pitch_initial)"
+    right_elbow_pitch_initial="$(arg right_elbow_pitch_initial)"
+    right_wrist_pitch_initial="$(arg right_wrist_pitch_initial)"
+    right_wrist_roll_initial="$(arg right_wrist_roll_initial)"
+    right_gripper_initial="$(arg right_gripper_initial)"/>
 </robot>

File: ros2_ws/src/cleany_description/urdf/cleany_geometry.xacro (robot description, xacro)
@@ -2,5 +2,8 @@
   <xacro:include filename="$(find cleany_description)/urdf/physical_properties.xacro" />
   <xacro:include filename="$(find cleany_description)/urdf/dual_arm.xacro" />
+  <xacro:include filename="$(find cleany_description)/urdf/head_camera.xacro" />
   <xacro:macro name="cleany_robot_geometry" params="include_wheel_joints:=false">
+    <!-- Fixed mast belongs to every model, including the controller's TF tree. -->
+    <xacro:cleany_head_mount/>
     <link name="base_link">
       <xacro:cleany_link_properties link_name="base_link" />

File: ros2_ws/src/cleany_description/urdf/cleany_mujoco_ros2_control.xacro (robot description, xacro)
@@ -1,17 +1,17 @@
 <?xml version="1.0"?>
 <robot xmlns:xacro="http://www.ros.org/wiki/xacro">
-  <xacro:macro name="cleany_mujoco_arm_joint" params="joint_name">
+  <xacro:macro name="cleany_mujoco_arm_joint" params="joint_name initial_value">
     <joint name="${joint_name}">
       <command_interface name="position"/>
       <state_interface name="position">
-        <param name="initial_value">0.0</param>
+        <param name="initial_value">${initial_value}</param>
       </state_interface>
       <state_interface name="velocity"/>
     </joint>
   </xacro:macro>
-  <xacro:macro name="cleany_mujoco_read_only_joint" params="joint_name">
+  <xacro:macro name="cleany_mujoco_read_only_joint" params="joint_name initial_value">
     <joint name="${joint_name}">
       <state_interface name="position">
-        <param name="initial_value">0.0</param>
+        <param name="initial_value">${initial_value}</param>
       </state_interface>
       <state_interface name="velocity"/>
@@ -20,12 +20,18 @@
   <xacro:macro
     name="cleany_mujoco_ros2_control"
-    params="mujoco_model headless sim_speed_factor camera_publish_rate camera_name camera_frame_name enable_gripper_command">
+    params="mujoco_model headless sim_speed_factor camera_publish_rate camera_name camera_frame_name enable_gripper_command
+            left_shoulder_yaw_initial left_shoulder_pitch_initial left_elbow_pitch_initial left_wrist_pitch_initial left_wrist_roll_initial left_gripper_initial
+            right_shoulder_yaw_initial right_shoulder_pitch_initial right_elbow_pitch_initial right_wrist_pitch_initial right_wrist_roll_initial right_gripper_initial
+            hardware_plugin:=mujoco_ros2_control/MujocoSystemInterface scheduled_cameras:=false">
     <ros2_control name="MujocoSystem" type="system">
       <hardware>
-        <plugin>mujoco_ros2_control/MujocoSystemInterface</plugin>
+        <plugin>${hardware_plugin}</plugin>
         <param name="mujoco_model">${mujoco_model}</param>
         <param name="headless">${headless}</param>
         <param name="sim_speed_factor">${sim_speed_factor}</param>
         <param name="camera_publish_rate">${camera_publish_rate}</param>
+        <xacro:if value="${scheduled_cameras}">
+          <param name="scheduled_cameras">true</param>
+        </xacro:if>
         <param name="initial_keyframe">handeye_ros2_control_home</param>
       </hardware>
@@ -38,21 +44,21 @@
         <param name="depth_topic">/${camera_name}/depth</param>
       </sensor>
-      <xacro:cleany_mujoco_arm_joint joint_name="left_shoulder_yaw_joint"/>
-      <xacro:cleany_mujoco_arm_joint joint_name="left_shoulder_pitch_joint"/>
-      <xacro:cleany_mujoco_arm_joint joint_name="left_elbow_pitch_joint"/>
-      <xacro:cleany_mujoco_arm_joint joint_name="left_wrist_pitch_joint"/>
-      <xacro:cleany_mujoco_arm_joint joint_name="left_wrist_roll_joint"/>
-      <xacro:cleany_mujoco_arm_joint joint_name="right_shoulder_yaw_joint"/>
-      <xacro:cleany_mujoco_arm_joint joint_name="right_shoulder_pitch_joint"/>
-      <xacro:cleany_mujoco_arm_joint joint_name="right_elbow_pitch_joint"/>
-      <xacro:cleany_mujoco_arm_joint joint_name="right_wrist_pitch_joint"/>
-      <xacro:cleany_mujoco_arm_joint joint_name="right_wrist_roll_joint"/>
+      <xacro:cleany_mujoco_arm_joint joint_name="left_shoulder_yaw_joint" initial_value="${left_shoulder_yaw_initial}"/>
+      <xacro:cleany_mujoco_arm_joint joint_name="left_shoulder_pitch_joint" initial_value="${left_shoulder_pitch_initial}"/>
+      <xacro:cleany_mujoco_arm_joint joint_name="left_elbow_pitch_joint" initial_value="${left_elbow_pitch_initial}"/>
+      <xacro:cleany_mujoco_arm_joint joint_name="left_wrist_pitch_joint" initial_value="${left_wrist_pitch_initial}"/>
+      <xacro:cleany_mujoco_arm_joint joint_name="left_wrist_roll_joint" initial_value="${left_wrist_roll_initial}"/>
+      <xacro:cleany_mujoco_arm_joint joint_name="right_shoulder_yaw_joint" initial_value="${right_shoulder_yaw_initial}"/>
+      <xacro:cleany_mujoco_arm_joint joint_name="right_shoulder_pitch_joint" initial_value="${right_shoulder_pitch_initial}"/>
+      <xacro:cleany_mujoco_arm_joint joint_name="right_elbow_pitch_joint" initial_value="${right_elbow_pitch_initial}"/>
+      <xacro:cleany_mujoco_arm_joint joint_name="right_wrist_pitch_joint" initial_value="${right_wrist_pitch_initial}"/>
+      <xacro:cleany_mujoco_arm_joint joint_name="right_wrist_roll_joint" initial_value="${right_wrist_roll_initial}"/>
       <xacro:if value="${enable_gripper_command}">
-        <xacro:cleany_mujoco_arm_joint joint_name="left_gripper_joint"/>
-        <xacro:cleany_mujoco_arm_joint joint_name="right_gripper_joint"/>
+        <xacro:cleany_mujoco_arm_joint joint_name="left_gripper_joint" initial_value="${left_gripper_initial}"/>
+        <xacro:cleany_mujoco_arm_joint joint_name="right_gripper_joint" initial_value="${right_gripper_initial}"/>
       </xacro:if>
       <xacro:unless value="${enable_gripper_command}">
-        <xacro:cleany_mujoco_read_only_joint joint_name="left_gripper_joint"/>
-        <xacro:cleany_mujoco_read_only_joint joint_name="right_gripper_joint"/>
+        <xacro:cleany_mujoco_read_only_joint joint_name="left_gripper_joint" initial_value="${left_gripper_initial}"/>
+        <xacro:cleany_mujoco_read_only_joint joint_name="right_gripper_joint" initial_value="${right_gripper_initial}"/>
       </xacro:unless>
     </ros2_control>

File: ros2_ws/src/cleany_description/urdf/physical_properties.xacro (robot description, xacro)
@@ -630,4 +630,10 @@
         </material>
       </visual>
+      <collision name="mjcf_geom_71_0_self_filter_collision">
+        <origin xyz="4.08954814457e-12 1.5600333525e-12 -1.16272394365e-06" rpy="2.65358979332e-06 -3.35582256428e-13 9.74717818498e-12" />
+        <geometry>
+          <mesh filename="package://cleany_description/meshes/Fixed_Jaw_Motor.stl" scale="1 1 1" />
+        </geometry>
+      </collision>
       <collision name="mjcf_geom_72_0_collision">
         <origin xyz="4.08954944561e-12 1.56000906637e-12 -1.16272394366e-06" rpy="2.6535897933e-06 -3.35547845291e-13 9.74717868076e-12" />
@@ -651,4 +657,10 @@
         </material>
       </visual>
+      <collision name="mjcf_geom_78_0_self_filter_collision">
+        <origin xyz="5.51022591132e-08 -0.00699996818156 0.0239988737994" rpy="1.57079632677 6.32679579342e-06 -1.57079999999" />
+        <geometry>
+          <mesh filename="package://cleany_description/meshes/XLeRobot_camera1.stl" scale="0.001 0.001 0.001" />
+        </geometry>
+      </collision>
       <visual name="mjcf_geom_79_0_visual">
         <origin xyz="5.51022591513e-08 -0.00699996818156 0.0239988737994" rpy="1.57079632677 6.3267957937e-06 -1.57079999999" />
@@ -660,4 +672,10 @@
         </material>
       </visual>
+      <collision name="mjcf_geom_79_0_self_filter_collision">
+        <origin xyz="5.51022591513e-08 -0.00699996818156 0.0239988737994" rpy="1.57079632677 6.3267957937e-06 -1.57079999999" />
+        <geometry>
+          <mesh filename="package://cleany_description/meshes/XLeRobot_camera2.stl" scale="0.001 0.001 0.001" />
+        </geometry>
+      </collision>
     </xacro:if>
     <xacro:if value="${link_name == 'left_moving_jaw_link'}">
@@ -906,4 +924,10 @@
         </material>
       </visual>
+      <collision name="mjcf_geom_103_0_self_filter_collision">
+        <origin xyz="-1.75451667084e-13 1.72466207982e-14 -1.57319893348e-09" rpy="3.58979298692e-09 -3.3556837864e-13 1.31342831277e-14" />
+        <geometry>
+          <mesh filename="package://cleany_description/meshes/Fixed_Jaw_Motor.stl" scale="1 1 1" />
+        </geometry>
+      </collision>
       <collision name="mjcf_geom_104_0_collision">
         <origin xyz="-1.75492433085e-13 1.71772318591e-14 -1.57319893063e-09" rpy="3.58979317055e-09 -3.35534912368e-13 1.32416268892e-14" />
@@ -927,4 +951,10 @@
         </material>
       </visual>
+      <collision name="mjcf_geom_110_0_self_filter_collision">
+        <origin xyz="5.50979259921e-08 -0.00599990458298 0.0240000535035" rpy="1.57079632678 3.676795793e-06 -1.5708" />
+        <geometry>
+          <mesh filename="package://cleany_description/meshes/XLeRobot_camera1.stl" scale="0.001 0.001 0.001" />
+        </geometry>
+      </collision>
       <visual name="mjcf_geom_111_0_visual">
         <origin xyz="5.50979259431e-08 -0.00599990458298 0.0240000535035" rpy="1.57079632678 3.67679579317e-06 -1.5708" />
@@ -936,4 +966,10 @@
         </material>
       </visual>
+      <collision name="mjcf_geom_111_0_self_filter_collision">
+        <origin xyz="5.50979259431e-08 -0.00599990458298 0.0240000535035" rpy="1.57079632678 3.67679579317e-06 -1.5708" />
+        <geometry>
+          <mesh filename="package://cleany_description/meshes/XLeRobot_camera2.stl" scale="0.001 0.001 0.001" />
+        </geometry>
+      </collision>
     </xacro:if>
     <xacro:if value="${link_name == 'right_moving_jaw_link'}">

Commit message: fix(sim): optimize MuJoCo rendering and recover wrist detection misses

File: ros2_ws/src/cleany_description/urdf/cleany_control.urdf.xacro (robot description, xacro)
@@ -7,4 +7,5 @@
   <xacro:arg name="camera_publish_rate" default="10.0"/>
   <xacro:arg name="scheduled_cameras" default="false"/>
+  <xacro:arg name="efficient_viewer" default="false"/>
   <xacro:arg name="camera_name" default="left_wrist_rgb"/>
   <xacro:arg name="camera_frame_name" default="left_wrist_rgb_vendor_frame"/>
@@ -33,4 +34,5 @@
     camera_publish_rate="$(arg camera_publish_rate)"
     scheduled_cameras="$(arg scheduled_cameras)"
+    efficient_viewer="$(arg efficient_viewer)"
     camera_name="$(arg camera_name)"
     camera_frame_name="$(arg camera_frame_name)"

File: ros2_ws/src/cleany_description/urdf/cleany_geometry.xacro (robot description, xacro)
@@ -9,6 +9,8 @@
       <xacro:cleany_link_properties link_name="base_link" />
     </link>
-    <xacro:cleany_arm side="left" side_sign="1" base_xyz="0.1163 0.185117 0.447797" base_yaw="3.14159265359" />
-    <xacro:cleany_arm side="right" side_sign="-1" base_xyz="0.116101 -0.185063 0.447797" base_yaw="0" />
+    <!-- Shoulder origins follow the CAD fastener-aligned Base placements in
+         physical_properties.xacro and mjcf/cleany.xml (see README). -->
+    <xacro:cleany_arm side="left" side_sign="1" base_xyz="0.116200343 0.196231727 0.447797" base_yaw="3.14159265359" />
+    <xacro:cleany_arm side="right" side_sign="-1" base_xyz="0.116200838 -0.196177072 0.447797" base_yaw="0" />
     <link name="rear_left_wheel_link">
       <xacro:cleany_link_properties link_name="rear_left_wheel_link" />

File: ros2_ws/src/cleany_description/urdf/cleany_mujoco_ros2_control.xacro (robot description, xacro)
@@ -23,5 +23,5 @@
             left_shoulder_yaw_initial left_shoulder_pitch_initial left_elbow_pitch_initial left_wrist_pitch_initial left_wrist_roll_initial left_gripper_initial
             right_shoulder_yaw_initial right_shoulder_pitch_initial right_elbow_pitch_initial right_wrist_pitch_initial right_wrist_roll_initial right_gripper_initial
-            hardware_plugin:=mujoco_ros2_control/MujocoSystemInterface scheduled_cameras:=false">
+            hardware_plugin:=mujoco_ros2_control/MujocoSystemInterface scheduled_cameras:=false efficient_viewer:=false">
     <ros2_control name="MujocoSystem" type="system">
       <hardware>
@@ -31,4 +31,5 @@
         <param name="sim_speed_factor">${sim_speed_factor}</param>
         <param name="camera_publish_rate">${camera_publish_rate}</param>
+        <param name="efficient_viewer">${str(efficient_viewer).lower()}</param>
         <xacro:if value="${scheduled_cameras}">
           <param name="scheduled_cameras">true</param>

File: ros2_ws/src/cleany_description/urdf/physical_properties.xacro (robot description, xacro)
@@ -2,8 +2,9 @@
   <xacro:macro name="cleany_link_properties" params="link_name">
     <xacro:if value="${link_name == 'base_link'}">
+      <!-- Combined chassis and fixed arm-base inertia at the aligned mounts. -->
       <inertial>
-        <origin xyz="0.00644072910811 2.68920880351e-05 -0.141372186369" rpy="0 -0 0" />
+        <origin xyz="0.00644073126036 2.68998835469e-05 -0.141372186369" rpy="0 -0 0" />
         <mass value="12.3513377764" />
-        <inertia ixx="0.932591878949" ixy="0.0005589332157" ixz="-0.046314226328" iyy="0.865628944375" iyz="1.45840680831e-08" izz="0.486831237121" />
+        <inertia ixx="0.933542754865" ixy="0.000607852427179" ixz="-0.0463142424415" iyy="0.865629751875" iyz="-4.37794203494e-08" izz="0.487782920537" />
       </inertial>
       <visual name="mjcf_geom_0_0_visual">
@@ -379,6 +380,7 @@
         </geometry>
       </collision>
+      <!-- Base/Motor visual and collision poses share the CAD mounting-hole fit. -->
       <visual name="mjcf_geom_48_0_visual">
-        <origin xyz="0.1163 0.139917 0.431297" rpy="0 -0 3.14159265359" />
+        <origin xyz="0.116200343 0.151031727 0.431297" rpy="0 -0 3.14159265359" />
         <geometry>
           <mesh filename="package://cleany_description/meshes/Base.stl" scale="1 1 1" />
@@ -389,5 +391,5 @@
       </visual>
       <visual name="mjcf_geom_49_0_visual">
-        <origin xyz="0.1163 0.139917 0.431297" rpy="0 -0 3.14159265359" />
+        <origin xyz="0.116200343 0.151031727 0.431297" rpy="0 -0 3.14159265359" />
         <geometry>
           <mesh filename="package://cleany_description/meshes/Base_Motor.stl" scale="1 1 1" />
@@ -398,5 +400,5 @@
       </visual>
       <collision name="mjcf_geom_50_0_collision">
-        <origin xyz="0.1163 0.139917 0.431297" rpy="0 -0 3.14159265359" />
+        <origin xyz="0.116200343 0.151031727 0.431297" rpy="0 -0 3.14159265359" />
         <geometry>
           <mesh filename="package://cleany_description/meshes/Base.stl" scale="1 1 1" />
@@ -404,5 +406,5 @@
       </collision>
       <collision name="mjcf_geom_51_0_collision">
-        <origin xyz="0.1163 0.139917 0.431297" rpy="0 -0 3.14159265359" />
+        <origin xyz="0.116200343 0.151031727 0.431297" rpy="0 -0 3.14159265359" />
         <geometry>
           <mesh filename="package://cleany_description/meshes/Base_Motor.stl" scale="1 1 1" />
@@ -410,5 +412,5 @@
       </collision>
       <visual name="mjcf_geom_80_0_visual">
-        <origin xyz="0.116101000162 -0.139863 0.431297" rpy="0 -5.55111512313e-17 -3.58979312866e-09" />
+        <origin xyz="0.116200838 -0.150977072 0.431297" rpy="0 -5.55111512313e-17 -3.58979312866e-09" />
         <geometry>
           <mesh filename="package://cleany_description/meshes/Base.stl" scale="1 1 1" />
@@ -419,5 +421,5 @@
       </visual>
       <visual name="mjcf_geom_81_0_visual">
-        <origin xyz="0.116101000162 -0.139863 0.431297" rpy="0 -0 -3.58979302984e-09" />
+        <origin xyz="0.116200838 -0.150977072 0.431297" rpy="0 -0 -3.58979302984e-09" />
         <geometry>
           <mesh filename="package://cleany_description/meshes/Base_Motor.stl" scale="1 1 1" />
@@ -428,5 +430,5 @@
       </visual>
       <collision name="mjcf_geom_82_0_collision">
-        <origin xyz="0.116101000162 -0.139863 0.431297" rpy="0 -5.55111512313e-17 -3.58979312866e-09" />
+        <origin xyz="0.116200838 -0.150977072 0.431297" rpy="0 -5.55111512313e-17 -3.58979312866e-09" />
         <geometry>
           <mesh filename="package://cleany_description/meshes/Base.stl" scale="1 1 1" />
@@ -434,5 +436,5 @@
       </collision>
       <collision name="mjcf_geom_83_0_collision">
-        <origin xyz="0.116101000162 -0.139863 0.431297" rpy="0 -0 -3.58979302984e-09" />
+        <origin xyz="0.116200838 -0.150977072 0.431297" rpy="0 -0 -3.58979302984e-09" />
         <geometry>
           <mesh filename="package://cleany_description/meshes/Base_Motor.stl" scale="1 1 1" />
