Commit message: feat(model): migrate dual-arm CAD geometry and five-axis chains

File: ros2_ws/src/cleany_description/urdf/cad_v1.urdf (robot description, URDF)
Before this commit: robot cleany, 5 links, 4 joints
Links:
- added link left_base_link, mass 0.15; visual mesh filename=package://cleany_description/meshes/cad_v1/left_base_printe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; visual mesh filename=package://cleany_description/meshes/cad_v1/left_base_servo.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
- added link left_gripper_frame, mass 0.25; visual mesh filename=package://cleany_description/meshes/cad_v1/left_tool_printe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; visual mesh filename=package://cleany_description/meshes/cad_v1/left_tool_servo.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
- added link left_lower_arm_link, mass 0.22; visual mesh filename=package://cleany_description/meshes/cad_v1/left_lower_carbo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; visual mesh filename=package://cleany_description/meshes/cad_v1/left_lower_print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
- added link left_shoulder_yaw_link, mass 0.22; visual mesh filename=package://cleany_description/meshes/cad_v1/left_yaw_printed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; visual mesh filename=package://cleany_description/meshes/cad_v1/left_yaw_servo.s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
- added link left_upper_arm_link, mass 0.22; visual mesh filename=package://cleany_description/meshes/cad_v1/left_upper_carbo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; visual mesh filename=package://cleany_description/meshes/cad_v1/left_upper_print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
- added link left_wrist_pitch_link, mass 0.22; visual mesh filename=package://cleany_description/meshes/cad_v1/left_wrist_print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; visual mesh filename=package://cleany_description/meshes/cad_v1/left_wrist_servo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
- added link right_base_link, mass 0.15; visual mesh filename=package://cleany_description/meshes/cad_v1/right_base_print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; visual mesh filename=package://cleany_description/meshes/cad_v1/right_base_servo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
- added link right_gripper_frame, mass 0.25; visual mesh filename=package://cleany_description/meshes/cad_v1/right_tool_print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; visual mesh filename=package://cleany_description/meshes/cad_v1/right_tool_servo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
- added link right_lower_arm_link, mass 0.22; visual mesh filename=package://cleany_description/meshes/cad_v1/right_lower_carb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; visual mesh filename=package://cleany_description/meshes/cad_v1/right_lower_prin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
- added link right_shoulder_yaw_link, mass 0.22; visual mesh filename=package://cleany_description/meshes/cad_v1/right_yaw_printe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; visual mesh filename=package://cleany_description/meshes/cad_v1/right_yaw_servo.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
- added link right_upper_arm_link, mass 0.22; visual mesh filename=package://cleany_description/meshes/cad_v1/right_upper_carb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; visual mesh filename=package://cleany_description/meshes/cad_v1/right_upper_prin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
- added link right_wrist_pitch_link, mass 0.22; visual mesh filename=package://cleany_description/meshes/cad_v1/right_wrist_prin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; visual mesh filename=package://cleany_description/meshes/cad_v1/right_wrist_serv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
Joints:
- added joint left_base_link_fixed: type fixed, parent base_link, child left_base_link, origin xyz=-0.12002511939 0.151030792567 0.331102994851 rpy=-7.33800009645e-09 5.55160004634e-08 -3.14158898038
- added joint left_elbow_pitch_joint: type revolute, parent left_upper_arm_link, child left_lower_arm_link, origin xyz=0 0.16257 0.028 rpy=1.57079632679 -0 3.14159265359, axis -1 0 0, limit lower=-0.22 upper=3.14 effort=4.41 velocity=4.245
- added joint left_shoulder_pitch_joint: type revolute, parent left_shoulder_yaw_link, child left_upper_arm_link, origin xyz=0 0.1025 0.0306 rpy=1.57079632679 -0 0, axis -1 0 0, limit lower=-0.22 upper=3.37 effort=4.41 velocity=4.245
- added joint left_shoulder_yaw_joint: type revolute, parent left_base_link, child left_shoulder_yaw_link, origin xyz=0 -0.0452 0.0165 rpy=1.57079632679 -0 0, axis 0 1 0, limit lower=-2.16 upper=2.16 effort=2.65 velocity=4.245
- added joint left_wrist_pitch_joint: type revolute, parent left_lower_arm_link, child left_wrist_pitch_link, origin xyz=0 -0.0052 0.1849 rpy=-1.57079632679 -0 0, axis 1 0 0, limit lower=-1.658063 upper=1.658063 effort=2.65 velocity=4.245
- added joint left_wrist_roll_joint: type revolute, parent left_wrist_pitch_link, child left_gripper_frame, origin xyz=-0.00152720656655 -0.05705 0 rpy=0 1.57079632679 -0, axis 0 -1 0, limit lower=-2.743847 upper=2.841206 effort=2.65 velocity=4.245
- added joint right_base_link_fixed: type fixed, parent base_link, child right_base_link, origin xyz=-0.12002401005 -0.150978005025 0.331102992634 rpy=7.33800009645e-09 -5.55160004634e-08 3.67320510257e-06
- added joint right_elbow_pitch_joint: type revolute, parent right_upper_arm_link, child right_lower_arm_link, origin xyz=0 0.16257 0.028 rpy=1.57079632679 -0 3.14159265359, axis -1 0 0, limit lower=-0.22 upper=3.14 effort=4.41 velocity=4.245
- added joint right_shoulder_pitch_joint: type revolute, parent right_shoulder_yaw_link, child right_upper_arm_link, origin xyz=0 0.1025 0.0306 rpy=1.57079632679 -0 0, axis -1 0 0, limit lower=-0.22 upper=3.37 effort=4.41 velocity=4.245
- added joint right_shoulder_yaw_joint: type revolute, parent right_base_link, child right_shoulder_yaw_link, origin xyz=0 -0.0452 0.0165 rpy=1.57079632679 -0 0, axis 0 1 0, limit lower=-2.16 upper=2.16 effort=2.65 velocity=4.245
- added joint right_wrist_pitch_joint: type revolute, parent right_lower_arm_link, child right_wrist_pitch_link, origin xyz=0 -0.0052 0.1849 rpy=-1.57079632679 -0 0, axis 1 0 0, limit lower=-1.658063 upper=1.658063 effort=2.65 velocity=4.245
- added joint right_wrist_roll_joint: type revolute, parent right_wrist_pitch_link, child right_gripper_frame, origin xyz=-0.00152720656655 -0.05705 0 rpy=0 1.57079632679 -0, axis 0 -1 0, limit lower=-2.743847 upper=2.841206 effort=2.65 velocity=4.245

Commit message: feat(model): add independent PincOpen closed-chain grippers

File: ros2_ws/src/cleany_description/urdf/cad_v1.urdf (robot description, URDF)
Before this commit: robot cleany, 17 links, 16 joints
Links:
- added link left_finger_1_distal, mass 0.028; visual mesh filename=package://cleany_description/meshes/cad_v1/left_finger_1_di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
- added link left_finger_1_driving, mass 0.006; visual mesh filename=package://cleany_description/meshes/cad_v1/left_finger_1_dr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
- added link left_finger_1_external, mass 0.008; visual mesh filename=package://cleany_description/meshes/cad_v1/left_finger_1_ex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
- added link left_finger_1_internal, mass 0.018; visual mesh filename=package://cleany_description/meshes/cad_v1/left_finger_1_in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
- added link left_finger_2_distal, mass 0.028; visual mesh filename=package://cleany_description/meshes/cad_v1/left_finger_2_di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
- added link left_finger_2_driving, mass 0.006; visual mesh filename=package://cleany_description/meshes/cad_v1/left_finger_2_dr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
- added link left_finger_2_external, mass 0.008; visual mesh filename=package://cleany_description/meshes/cad_v1/left_finger_2_ex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
- added link left_finger_2_internal, mass 0.018; visual mesh filename=package://cleany_description/meshes/cad_v1/left_finger_2_in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
- added link left_grasp_tcp
- added link left_gripper_cam_link, mass 0.012; visual mesh filename=package://cleany_description/meshes/cad_v1/left_cam.stl
- added link left_pregrasp_aim_tip
- added link right_finger_1_distal, mass 0.028; visual mesh filename=package://cleany_description/meshes/cad_v1/right_finger_1_d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
- added link right_finger_1_driving, mass 0.006; visual mesh filename=package://cleany_description/meshes/cad_v1/right_finger_1_d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
- added link right_finger_1_external, mass 0.008; visual mesh filename=package://cleany_description/meshes/cad_v1/right_finger_1_e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
- added link right_finger_1_internal, mass 0.018; visual mesh filename=package://cleany_description/meshes/cad_v1/right_finger_1_i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
- added link right_finger_2_distal, mass 0.028; visual mesh filename=package://cleany_description/meshes/cad_v1/right_finger_2_d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
- added link right_finger_2_driving, mass 0.006; visual mesh filename=package://cleany_description/meshes/cad_v1/right_finger_2_d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
- added link right_finger_2_external, mass 0.008; visual mesh filename=package://cleany_description/meshes/cad_v1/right_finger_2_e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
- added link right_finger_2_internal, mass 0.018; visual mesh filename=package://cleany_description/meshes/cad_v1/right_finger_2_i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
- added link right_grasp_tcp
- added link right_gripper_cam_link, mass 0.012; visual mesh filename=package://cleany_description/meshes/cad_v1/right_cam.stl
- added link right_pregrasp_aim_tip
- link left_gripper_frame: mass 0.25 -> 0.13; geometry visual mesh filename=package://cleany_description/meshes/cad_v1/left_palm.stl
- link right_gripper_frame: mass 0.25 -> 0.13; geometry visual mesh filename=package://cleany_description/meshes/cad_v1/right_palm.stl
Joints:
- added joint left_finger_1_distal_joint: type revolute, parent left_finger_1_internal, child left_finger_1_distal, origin xyz=0.0346410161514 0.02 0 rpy=0 -0 0, axis 0 0 1, limit lower=-3.141592653589793 upper=3.141592653589793 effort=2.65 velocity=4.245
- added joint left_finger_1_driving_joint: type revolute, parent left_gripper_cam_link, child left_finger_1_driving, origin xyz=-0.00354167484447 -0.0104142469388 0 rpy=0 -0 0, axis 0 0 1, limit lower=-3.141592653589793 upper=3.141592653589793 effort=2.65 velocity=4.245
- added joint left_finger_1_external_joint: type revolute, parent left_gripper_frame, child left_finger_1_external, origin xyz=0 -0.0671089838486 0.044 rpy=-1.57079632679 -0 -1.57079632679, axis 0 0 1, limit lower=-3.141592653589793 upper=3.141592653589793 effort=2.65 velocity=4.245
- added joint left_finger_1_internal_joint: type revolute, parent left_gripper_frame, child left_finger_1_internal, origin xyz=0 -0.0671089838486 0.0325 rpy=-1.57079632679 -0 -1.57079632679, axis 0 0 1, limit lower=-3.141592653589793 upper=3.141592653589793 effort=2.65 velocity=4.245
- added joint left_finger_2_distal_joint: type revolute, parent left_finger_2_internal, child left_finger_2_distal, origin xyz=0.0346410161514 -0.02 0 rpy=0 -0 0, axis 0 0 1, limit lower=-3.141592653589793 upper=3.141592653589793 effort=2.65 velocity=4.245
- added joint left_finger_2_driving_joint: type revolute, parent left_gripper_cam_link, child left_finger_2_driving, origin xyz=0.00330082918453 0.01049307041 0 rpy=0 -0 0, axis 0 0 1, limit lower=-3.141592653589793 upper=3.141592653589793 effort=2.65 velocity=4.245
- added joint left_finger_2_external_joint: type revolute, parent left_gripper_frame, child left_finger_2_external, origin xyz=0 -0.0671089838486 -0.044 rpy=-1.57079632679 -0 -1.57079632679, axis 0 0 1, limit lower=-3.141592653589793 upper=3.141592653589793 effort=2.65 velocity=4.245
- added joint left_finger_2_internal_joint: type revolute, parent left_gripper_frame, child left_finger_2_internal, origin xyz=0 -0.0671089838486 -0.0325 rpy=-1.57079632679 -0 -1.57079632679, axis 0 0 1, limit lower=-3.141592653589793 upper=3.141592653589793 effort=2.65 velocity=4.245
- added joint left_grasp_tcp_fixed: type fixed, parent left_gripper_frame, child left_grasp_tcp, origin xyz=0 -0.119132450457 0 rpy=-1.57079632679 -0 -1.57079632679
- added joint left_gripper_joint: type revolute, parent left_gripper_frame, child left_gripper_cam_link, origin xyz=0 -0.0490665820841 0 rpy=-1.57079632679 -0 -1.57079632679, axis 0 0 1, limit lower=-1.0471975511965976 upper=0 effort=1.5 velocity=4.245
- added joint left_pregrasp_aim_tip_fixed: type fixed, parent left_gripper_frame, child left_pregrasp_aim_tip, origin xyz=0 -0.259132450457 0 rpy=-1.57079632679 -0 -1.57079632679
- added joint right_finger_1_distal_joint: type revolute, parent right_finger_1_internal, child right_finger_1_distal, origin xyz=0.0346410161514 0.02 0 rpy=0 -0 0, axis 0 0 1, limit lower=-3.141592653589793 upper=3.141592653589793 effort=2.65 velocity=4.245
- added joint right_finger_1_driving_joint: type revolute, parent right_gripper_cam_link, child right_finger_1_driving, origin xyz=-0.00354167484447 -0.0104142469388 0 rpy=0 -0 0, axis 0 0 1, limit lower=-3.141592653589793 upper=3.141592653589793 effort=2.65 velocity=4.245
- added joint right_finger_1_external_joint: type revolute, parent right_gripper_frame, child right_finger_1_external, origin xyz=0 -0.0671089838486 0.044 rpy=-1.57079632679 -0 -1.57079632679, axis 0 0 1, limit lower=-3.141592653589793 upper=3.141592653589793 effort=2.65 velocity=4.245
- added joint right_finger_1_internal_joint: type revolute, parent right_gripper_frame, child right_finger_1_internal, origin xyz=0 -0.0671089838486 0.0325 rpy=-1.57079632679 -0 -1.57079632679, axis 0 0 1, limit lower=-3.141592653589793 upper=3.141592653589793 effort=2.65 velocity=4.245
- added joint right_finger_2_distal_joint: type revolute, parent right_finger_2_internal, child right_finger_2_distal, origin xyz=0.0346410161514 -0.02 0 rpy=0 -0 0, axis 0 0 1, limit lower=-3.141592653589793 upper=3.141592653589793 effort=2.65 velocity=4.245
- added joint right_finger_2_driving_joint: type revolute, parent right_gripper_cam_link, child right_finger_2_driving, origin xyz=0.00330082918453 0.01049307041 0 rpy=0 -0 0, axis 0 0 1, limit lower=-3.141592653589793 upper=3.141592653589793 effort=2.65 velocity=4.245
- added joint right_finger_2_external_joint: type revolute, parent right_gripper_frame, child right_finger_2_external, origin xyz=0 -0.0671089838486 -0.044 rpy=-1.57079632679 -0 -1.57079632679, axis 0 0 1, limit lower=-3.141592653589793 upper=3.141592653589793 effort=2.65 velocity=4.245
- added joint right_finger_2_internal_joint: type revolute, parent right_gripper_frame, child right_finger_2_internal, origin xyz=0 -0.0671089838486 -0.0325 rpy=-1.57079632679 -0 -1.57079632679, axis 0 0 1, limit lower=-3.141592653589793 upper=3.141592653589793 effort=2.65 velocity=4.245
- added joint right_grasp_tcp_fixed: type fixed, parent right_gripper_frame, child right_grasp_tcp, origin xyz=0 -0.119132450457 0 rpy=-1.57079632679 -0 -1.57079632679
- added joint right_gripper_joint: type revolute, parent right_gripper_frame, child right_gripper_cam_link, origin xyz=0 -0.0490665820841 0 rpy=-1.57079632679 -0 -1.57079632679, axis 0 0 1, limit lower=-1.0471975511965976 upper=0 effort=1.5 velocity=4.245
- added joint right_pregrasp_aim_tip_fixed: type fixed, parent right_gripper_frame, child right_pregrasp_aim_tip, origin xyz=0 -0.259132450457 0 rpy=-1.57079632679 -0 -1.57079632679

Commit message: feat(model): migrate head wrist cameras lidar and IMU

File: ros2_ws/src/cleany_description/urdf/cad_v1.urdf (robot description, URDF)
Before this commit: robot cleany, 39 links, 38 joints
Links:
- added link head_camera_depth_frame
- added link head_camera_depth_optical_frame
- added link head_camera_link
- added link head_camera_rgb_frame
- added link head_camera_rgb_optical_frame
- added link head_pan_link, mass 0.1; visual mesh filename=package://cleany_description/meshes/cad_v1/head_pan_hardwar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; visual mesh filename=package://cleany_description/meshes/cad_v1/head_pan_plastic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
- added link head_tilt_link, mass 0.12; visual mesh filename=package://cleany_description/meshes/cad_v1/head_tilt_camera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; visual mesh filename=package://cleany_description/meshes/cad_v1/head_tilt_hardwa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
- added link imu_link, mass 0.035; visual mesh filename=package://cleany_description/meshes/cad_v1/imuboardbolts.stl; visual mesh filename=package://cleany_description/meshes/cad_v1/imuboardnuts.stl
- added link imu_site
- added link laser
- added link left_wrist_camera_link, mass 0.065; visual mesh filename=package://cleany_description/meshes/cad_v1/left_camera_hard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; visual mesh filename=package://cleany_description/meshes/cad_v1/left_camera_moun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
- added link left_wrist_rgb_optical_frame
- added link lidar_link, mass 0.25; visual mesh filename=package://cleany_description/meshes/cad_v1/lidarlowerbolts.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; visual mesh filename=package://cleany_description/meshes/cad_v1/lidarplate.stl
- added link lidar_site
- added link right_wrist_camera_link, mass 0.065; visual mesh filename=package://cleany_description/meshes/cad_v1/right_camera_har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; visual mesh filename=package://cleany_description/meshes/cad_v1/right_camera_mou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
- added link right_wrist_rgb_optical_frame
- added link top_base_link, mass 0.09; visual mesh filename=package://cleany_description/meshes/cad_v1/head_base_plasti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; visual mesh filename=package://cleany_description/meshes/cad_v1/head_base_servo.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
Joints:
- added joint head_camera_depth_frame_fixed: type fixed, parent head_tilt_link, child head_camera_depth_frame, origin xyz=0.0355500000024 -1.86517468137e-17 0.0323960780542 rpy=2.22044604925e-16 1.11022302463e-16 2.22044604925e-16
- added joint head_camera_depth_optical_frame_fixed: type fixed, parent head_tilt_link, child head_camera_depth_optical_frame, origin xyz=0.0355500000024 -1.86517468137e-17 0.0323960780542 rpy=-1.57079632679 1.57009245868e-16 -1.57079632679
- added joint head_camera_link_fixed: type fixed, parent head_tilt_link, child head_camera_link, origin xyz=0.0355500000024 -1.86517468137e-17 0.0323960780542 rpy=2.22044604925e-16 1.11022302463e-16 2.22044604925e-16
- added joint head_camera_rgb_frame_fixed: type fixed, parent head_tilt_link, child head_camera_rgb_frame, origin xyz=0.0355500000024 -1.86517468137e-17 0.0323960780542 rpy=2.22044604925e-16 1.11022302463e-16 2.22044604925e-16
- added joint head_camera_rgb_optical_frame_fixed: type fixed, parent head_tilt_link, child head_camera_rgb_optical_frame, origin xyz=0.0355500000024 -1.86517468137e-17 0.0323960780542 rpy=-1.57079632679 1.57009245868e-16 -1.57079632679
- added joint head_pan_joint: type revolute, parent top_base_link, child head_pan_link, origin xyz=-0.213473591202 0.0061 1.1169 rpy=0 -0 0, axis 0 0 1, limit lower=-1.5707963267948966 upper=1.5707963267948966 effort=2.65 velocity=4.245
- added joint head_tilt_joint: type revolute, parent head_pan_link, child head_tilt_link, origin xyz=1e-05 -0.0006 0.023375 rpy=0 -0 0, axis 0 1 0, limit lower=-0.7853981633974483 upper=0.7853981633974483 effort=2.65 velocity=4.245
- added joint imu_link_fixed: type fixed, parent base_link, child imu_link, origin xyz=-2.45388500298e-05 2.68379755866e-05 -0.134897 rpy=-7.33800009645e-09 5.55160004634e-08 -3.14158898038
- added joint imu_site_fixed: type fixed, parent imu_link, child imu_site, origin xyz=0 0 0 rpy=0 -0 0
- added joint laser_fixed: type fixed, parent lidar_link, child laser, origin xyz=0 0 0 rpy=0 -0 0
- added joint left_wrist_camera_link_fixed: type fixed, parent left_gripper_frame, child left_wrist_camera_link, origin xyz=0.066724675601 -0.0631437997693 2.53130849615e-17 rpy=0 1.57079632679 -2.44346095279
- added joint left_wrist_rgb_optical_frame_fixed: type fixed, parent left_wrist_camera_link, child left_wrist_rgb_optical_frame, origin xyz=0 0 0 rpy=0 -0 0
- added joint lidar_link_fixed: type fixed, parent base_link, child lidar_link, origin xyz=-0.139299541203 2.6326078806e-05 -0.092497007732 rpy=5.55160004634e-08 7.33800009645e-09 -1.57079265359
- added joint lidar_site_fixed: type fixed, parent lidar_link, child lidar_site, origin xyz=0 0 0 rpy=0 -0 0
- added joint right_wrist_camera_link_fixed: type fixed, parent right_gripper_frame, child right_wrist_camera_link, origin xyz=0.066724675601 -0.0631437997693 2.53130849615e-17 rpy=0 1.57079632679 -2.44346095279
- added joint right_wrist_rgb_optical_frame_fixed: type fixed, parent right_wrist_camera_link, child right_wrist_rgb_optical_frame, origin xyz=0 0 0 rpy=0 -0 0
- added joint top_base_link_fixed: type fixed, parent base_link, child top_base_link, origin xyz=-0.300915876239 0.00613319730702 -0.435385493097 rpy=-7.33800009645e-09 5.55160003524e-08 -3.14158898038
