Commit message: feat(model): add collision meshes inertias and contact physics

File: ros2_ws/src/cleany_description/urdf/cad_v1.urdf (robot description, URDF)
Before this commit: robot cleany, 56 links, 55 joints
Links:
- link base_link: mass 8.0 -> 8.465515123837198; geometry collision box size=0.0200000942178 0.0200000730196 0.440000001304; collision box size=0.0200000942178 0.0200000730196 0.440000001304
- link front_left_wheel_link: mass 0.38 -> .5; geometry collision cylinder length=.051 radius=.0635; visual mesh filename=package://cleany_description/meshes/cad_v1/front_left_wheel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
- link front_right_wheel_link: mass 0.38 -> .5; geometry collision cylinder length=.051 radius=.0635; visual mesh filename=package://cleany_description/meshes/cad_v1/front_right_whee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
- link head_pan_link: mass 0.1 -> 0.08198923533545688; geometry collision box size=0.0192 0.0192 0.00335; collision box size=0.0192 0.0192 0.0045000001
- link head_tilt_link: mass 0.12 -> 0.09733350074312185; geometry collision box size=0.011 0.0055000002 0.0055000002; collision box size=0.011 0.0055000002 0.0055000002
- link imu_link: mass 0.035 -> 0.018832047383362863; geometry collision box size=0.00254 0.02032 0.011; collision box size=0.004 0.004 0.0009
- link left_base_link: mass 0.15 -> 0.1501740431517099; geometry collision box size=0.0245000002 0.0450000002 0.0097000001; collision box size=0.0247200002 0.0452200002 0.0141000002013
- link left_finger_1_distal: mass 0.028 -> 0.00792952677678155; geometry collision box size=0.0070151 0.002 0.01038399; collision box size=0.0070151 0.002 0.01038399
- link left_finger_1_driving: mass 0.006 -> 0.0010740527364630176; geometry collision box size=0.016120476541 0.0425051542832 0.0053000002; visual mesh filename=package://cleany_description/meshes/cad_v1/left_finger_1_dr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
- link left_finger_1_external: mass 0.008 -> 0.002110236426275736; geometry collision box size=0.0436410161514 0.029 0.0080000002; visual mesh filename=package://cleany_description/meshes/cad_v1/left_finger_1_ex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
- link left_finger_1_internal: mass 0.018 -> 0.0036140700056098104; geometry collision mesh filename=package://cleany_description/meshes/cad_v1/finger_1_interna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; collision mesh filename=package://cleany_description/meshes/cad_v1/finger_1_interna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
- link left_finger_2_distal: mass 0.028 -> 0.00792952677678155; geometry collision box size=0.00350755 0.002 0.01038399; collision box size=0.00350755 0.002 0.01038399
- link left_finger_2_driving: mass 0.006 -> 0.0010740527364630171; geometry collision box size=0.0165609229483 0.0424263308087 0.0053000002; visual mesh filename=package://cleany_description/meshes/cad_v1/left_finger_2_dr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
- link left_finger_2_external: mass 0.008 -> 0.002110236426275736; geometry collision box size=0.0436410161514 0.029 0.0080000002; visual mesh filename=package://cleany_description/meshes/cad_v1/left_finger_2_ex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
- link left_finger_2_internal: mass 0.018 -> 0.00361407000560981; geometry collision mesh filename=package://cleany_description/meshes/cad_v1/finger_2_interna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; collision mesh filename=package://cleany_description/meshes/cad_v1/finger_2_interna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
- link left_gripper_cam_link: mass 0.012 -> 0.003467308184406045; geometry collision box size=0.0192000002 0.0192000002 0.0045000002; collision box size=0.0320078107936 0.0320000002 0.0068500002
- link left_gripper_frame: geometry collision box size=0.0097000001 0.0450000002 0.0245000002; collision box size=0.0139000002 0.0452234080154 0.0247234080154
- link left_lower_arm_link: mass 0.22 -> 0.11506178963183422; geometry collision box size=0.00335000257111 0.0192000002 0.0192000002; collision box size=0.0045000002 0.0192000002 0.0192000002
- link left_shoulder_yaw_link: mass 0.22 -> 0.10924200458409095; geometry collision box size=0.0097000001 0.0450000002 0.0245000002; collision box size=0.0139000002 0.0452234080154 0.0247234080154
- link left_upper_arm_link: mass 0.22 -> 0.11360422934603755; geometry collision box size=0.00335000257111 0.0192000002 0.0192000002; collision box size=0.0045000002 0.0192000002 0.0192000002
- link left_wrist_camera_link: mass 0.065 -> 0.042546690997913146; geometry collision box size=0.0038 0.0038 0.022; collision box size=0.0038 0.0038 0.022
- link left_wrist_pitch_link: mass 0.22 -> 0.07673142399116653; geometry collision box size=0.00335000257111 0.0192000002 0.0192000002; collision box size=0.0045000002 0.0192000002 0.0192000002
- link lidar_link: mass 0.25 -> 0.43242420154660005; geometry collision box size=0.003985 0.0042000001 0.0047; collision box size=0.003985 0.0042000001 0.0047
- link rear_left_wheel_link: mass 0.38 -> .5; geometry collision cylinder length=.051 radius=.0635; visual mesh filename=package://cleany_description/meshes/cad_v1/rear_left_wheel.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
- link rear_right_wheel_link: mass 0.38 -> .5; geometry collision cylinder length=.051 radius=.0635; visual mesh filename=package://cleany_description/meshes/cad_v1/rear_right_wheel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
- link right_base_link: mass 0.15 -> 0.1501740431517099; geometry collision box size=0.0245000002 0.0450000002 0.0097000001; collision box size=0.0247200002 0.0452200002 0.0141000002013
- link right_finger_1_distal: mass 0.028 -> 0.00792952677678155; geometry collision box size=0.0070151 0.002 0.01038399; collision box size=0.0070151 0.002 0.01038399
- link right_finger_1_driving: mass 0.006 -> 0.0010740527364630176; geometry collision box size=0.016120476541 0.0425051542832 0.0053000002; visual mesh filename=package://cleany_description/meshes/cad_v1/right_finger_1_d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
- link right_finger_1_external: mass 0.008 -> 0.002110236426275736; geometry collision box size=0.0436410161514 0.029 0.0080000002; visual mesh filename=package://cleany_description/meshes/cad_v1/right_finger_1_e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
- link right_finger_1_internal: mass 0.018 -> 0.0036140700056098104; geometry collision mesh filename=package://cleany_description/meshes/cad_v1/finger_1_interna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; collision mesh filename=package://cleany_description/meshes/cad_v1/finger_1_interna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
- link right_finger_2_distal: mass 0.028 -> 0.00792952677678155; geometry collision box size=0.00350755 0.002 0.01038399; collision box size=0.00350755 0.002 0.01038399
- link right_finger_2_driving: mass 0.006 -> 0.0010740527364630171; geometry collision box size=0.0165609229483 0.0424263308087 0.0053000002; visual mesh filename=package://cleany_description/meshes/cad_v1/right_finger_2_d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
- link right_finger_2_external: mass 0.008 -> 0.002110236426275736; geometry collision box size=0.0436410161514 0.029 0.0080000002; visual mesh filename=package://cleany_description/meshes/cad_v1/right_finger_2_e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
- link right_finger_2_internal: mass 0.018 -> 0.00361407000560981; geometry collision mesh filename=package://cleany_description/meshes/cad_v1/finger_2_interna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; collision mesh filename=package://cleany_description/meshes/cad_v1/finger_2_interna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
- link right_gripper_cam_link: mass 0.012 -> 0.003467308184406045; geometry collision box size=0.0192000002 0.0192000002 0.0045000002; collision box size=0.0320078107936 0.0320000002 0.0068500002
- link right_gripper_frame: geometry collision box size=0.0097000001 0.0450000002 0.0245000002; collision box size=0.0139000002 0.0452234080154 0.0247234080154
- link right_lower_arm_link: mass 0.22 -> 0.11506178963183422; geometry collision box size=0.00335000257111 0.0192000002 0.0192000002; collision box size=0.0045000002 0.0192000002 0.0192000002
- link right_shoulder_yaw_link: mass 0.22 -> 0.10924200458409095; geometry collision box size=0.0097000001 0.0450000002 0.0245000002; collision box size=0.0139000002 0.0452234080154 0.0247234080154
- link right_upper_arm_link: mass 0.22 -> 0.11360422934603755; geometry collision box size=0.00335000257111 0.0192000002 0.0192000002; collision box size=0.0045000002 0.0192000002 0.0192000002
- link right_wrist_camera_link: mass 0.065 -> 0.042546690997913146; geometry collision box size=0.0038 0.0038 0.022; collision box size=0.0038 0.0038 0.022
- link right_wrist_pitch_link: mass 0.22 -> 0.07673142399116653; geometry collision box size=0.00335000257111 0.0192000002 0.0192000002; collision box size=0.0045000002 0.0192000002 0.0192000002
- link top_base_link: mass 0.09 -> 0.08199726219358494; geometry collision box size=0.045 0.0245 0.0097000001; collision box size=0.0452200001 0.0247200002 0.0141000002

Commit message: feat(model): integrate CAD URDF Xacro and MuJoCo entrypoints

File: ros2_ws/src/cleany_description/urdf/cad_v1.urdf (robot description, URDF)
Before this commit: robot cleany, 56 links, 55 joints
Joints:
- joint left_gripper_joint: axis 0 0 1 -> 0 0 -1; limit lower=-1.0471975511965976 upper=0 effort=1.5 velocity=4.245 -> lower=0 upper=1.0471975511965976 effort=1.5 velocity=4.245
- joint right_gripper_joint: axis 0 0 1 -> 0 0 -1; limit lower=-1.0471975511965976 upper=0 effort=1.5 velocity=4.245 -> lower=0 upper=1.0471975511965976 effort=1.5 velocity=4.245

File: ros2_ws/src/cleany_description/urdf/cleany.urdf.xacro (robot description, xacro)
@@ -3,7 +3,7 @@
   <xacro:arg name="include_head_camera" default="true"/>
   <xacro:arg name="include_wheel_joints" default="true"/>
-  <xacro:include filename="$(find cleany_description)/urdf/materials.xacro"/>
-  <xacro:include filename="$(find cleany_description)/urdf/cleany_geometry.xacro"/>
-  <xacro:include filename="$(find cleany_description)/urdf/head_camera.xacro"/>
+  <xacro:include filename="materials.xacro"/>
+  <xacro:include filename="cleany_geometry.xacro"/>
+  <xacro:include filename="head_camera.xacro"/>
   <xacro:cleany_robot_geometry include_wheel_joints="$(arg include_wheel_joints)"/>
   <xacro:if value="$(arg include_head_camera)">

File: ros2_ws/src/cleany_description/urdf/cleany_control.urdf.xacro (robot description, xacro)
@@ -11,4 +11,5 @@
   <xacro:arg name="camera_frame_name" default="left_wrist_rgb_vendor_frame"/>
   <xacro:arg name="enable_gripper_command" default="false"/>
+  <xacro:arg name="include_head_camera" default="false"/>
   <xacro:arg name="left_shoulder_yaw_initial" default="0.0"/>
   <xacro:arg name="left_shoulder_pitch_initial" default="0.0"/>
@@ -23,8 +24,12 @@
   <xacro:arg name="right_wrist_roll_initial" default="0.0"/>
   <xacro:arg name="right_gripper_initial" default="0.0"/>
-  <xacro:include filename="$(find cleany_description)/urdf/materials.xacro"/>
-  <xacro:include filename="$(find cleany_description)/urdf/cleany_geometry.xacro"/>
-  <xacro:include filename="$(find cleany_description)/urdf/cleany_mujoco_ros2_control.xacro"/>
+  <xacro:include filename="materials.xacro"/>
+  <xacro:include filename="cleany_geometry.xacro"/>
+  <xacro:include filename="head_camera.xacro"/>
+  <xacro:include filename="cleany_mujoco_ros2_control.xacro"/>
   <xacro:cleany_robot_geometry/>
+  <xacro:if value="$(arg include_head_camera)">
+    <xacro:cleany_head_camera/>
+  </xacro:if>
   <xacro:cleany_mujoco_ros2_control
     mujoco_model="$(arg mujoco_model)"

File: ros2_ws/src/cleany_description/urdf/cleany_geometry.xacro (robot description, xacro)
@@ -1,56 +1,5 @@
+<?xml version="1.0"?>
 <robot xmlns:xacro="http://www.ros.org/wiki/xacro">
-  <xacro:include filename="$(find cleany_description)/urdf/physical_properties.xacro" />
-  <xacro:include filename="$(find cleany_description)/urdf/dual_arm.xacro" />
-  <xacro:include filename="$(find cleany_description)/urdf/head_camera.xacro" />
-  <xacro:macro name="cleany_robot_geometry" params="include_wheel_joints:=false">
-    <!-- Fixed mast belongs to every model, including the controller's TF tree. -->
-    <xacro:cleany_head_mount/>
-    <link name="base_link">
-      <xacro:cleany_link_properties link_name="base_link" />
-    </link>
-    <!-- Shoulder origins follow the CAD fastener-aligned Base placements in
-         physical_properties.xacro and mjcf/cleany.xml (see README). -->
-    <xacro:cleany_arm side="left" side_sign="1" base_xyz="0.116200343 0.196231727 0.447797" base_yaw="3.14159265359" />
-    <xacro:cleany_arm side="right" side_sign="-1" base_xyz="0.116200838 -0.196177072 0.447797" base_yaw="0" />
-    <link name="rear_left_wheel_link">
-      <xacro:cleany_link_properties link_name="rear_left_wheel_link" />
-    </link>
-    <joint name="rear_left_wheel_joint" type="${'continuous' if include_wheel_joints else 'fixed'}">
-      <origin xyz="-0.175025 0.301927 -0.316497" rpy="0 -0 0" />
-      <parent link="base_link" />
-      <child link="rear_left_wheel_link" />
-      <axis xyz="0 1 0" />
-      <limit effort="2.646" velocity="12.017" />
-    </joint>
-    <link name="rear_right_wheel_link">
-      <xacro:cleany_link_properties link_name="rear_right_wheel_link" />
-    </link>
-    <joint name="rear_right_wheel_joint" type="${'continuous' if include_wheel_joints else 'fixed'}">
-      <origin xyz="-0.175025 -0.301873 -0.316497" rpy="0 -0 0" />
-      <parent link="base_link" />
-      <child link="rear_right_wheel_link" />
-      <axis xyz="0 1 0" />
-      <limit effort="2.646" velocity="12.017" />
-    </joint>
-    <link name="front_left_wheel_link">
-      <xacro:cleany_link_properties link_name="front_left_wheel_link" />
-    </link>
-    <joint name="front_left_wheel_joint" type="${'continuous' if include_wheel_joints else 'fixed'}">
-      <origin xyz="0.174975 0.301927 -0.316497" rpy="0 -0 0" />
-      <parent link="base_link" />
-      <child link="front_left_wheel_link" />
-      <axis xyz="0 1 0" />
-      <limit effort="2.646" velocity="12.017" />
-    </joint>
-    <link name="front_right_wheel_link">
-      <xacro:cleany_link_properties link_name="front_right_wheel_link" />
-    </link>
-    <joint name="front_right_wheel_joint" type="${'continuous' if include_wheel_joints else 'fixed'}">
-      <origin xyz="0.174975 -0.301873 -0.316497" rpy="0 -0 0" />
-      <parent link="base_link" />
-      <child link="front_right_wheel_link" />
-      <axis xyz="0 1 0" />
-      <limit effort="2.646" velocity="12.017" />
-    </joint>
-  </xacro:macro>
+  <!-- Current CAD geometry; dimensions and joint origins use metres/radians. -->
+  <xacro:include filename="cad_v1_geometry.xacro"/>
 </robot>
