Commit message: fix(model): restore 140 degree PincOpen travel with fitted rod collisions

File: ros2_ws/src/cleany_description/urdf/cad_v1.urdf (robot description, URDF)
Before this commit: robot cleany, 56 links, 55 joints
Links:
- link left_finger_1_driving: geometry collision mesh filename=package://cleany_description/meshes/cad_v1/finger_1_driving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; collision mesh filename=package://cleany_description/meshes/cad_v1/finger_1_driving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
- link left_finger_2_driving: geometry collision mesh filename=package://cleany_description/meshes/cad_v1/finger_2_driving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; collision mesh filename=package://cleany_description/meshes/cad_v1/finger_2_driving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
- link right_finger_1_driving: geometry collision mesh filename=package://cleany_description/meshes/cad_v1/finger_1_driving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; collision mesh filename=package://cleany_description/meshes/cad_v1/finger_1_driving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
- link right_finger_2_driving: geometry collision mesh filename=package://cleany_description/meshes/cad_v1/finger_2_driving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; collision mesh filename=package://cleany_description/meshes/cad_v1/finger_2_driving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
Joints:
- joint left_gripper_joint: limit lower=0 upper=1.0471975511965976 effort=1.5 velocity=4.245 -> lower=0 upper=2.443460952792061 effort=1.5 velocity=4.245
- joint right_gripper_joint: limit lower=0 upper=1.0471975511965976 effort=1.5 velocity=4.245 -> lower=0 upper=2.443460952792061 effort=1.5 velocity=4.245

File: ros2_ws/src/cleany_description/urdf/cad_v1_geometry.xacro (robot description, xacro)
@@ -173,5 +173,5 @@
    limitations under the License.
 -->
-  <!--CAD source Cleany.FCStd SHA256 5fe6b78e2eb0ef183e66631eb8aef31503eb8f0b0c5902d9955affd8a7aef82e. Export units: metres and radians; visual tessellation 0.12 mm. Saved CAD folded pose is cad_home in cad_v1.xml. Public left/right follows REP-103 base +Y/-Y; CAD internal RightArm is ROS left. Positive gripper angle opens: 0 to pi/3 corresponds to source cam 0 to -60 degrees. Passive linkage joints require measured/simulated states; URDF mimic does not represent these nonlinear closed loops.-->
+  <!--CAD source Cleany.FCStd SHA256 5fe6b78e2eb0ef183e66631eb8aef31503eb8f0b0c5902d9955affd8a7aef82e. Export units: metres and radians; visual tessellation 0.12 mm. Saved CAD folded pose is cad_home in cad_v1.xml. Public left/right follows REP-103 base +Y/-Y; CAD internal RightArm is ROS left. Positive gripper angle opens: 0 to 2.443460952792061 radians corresponds to source cam 0 to -140 degrees (vendor v1.0 flash_test.ipynb open command; 147-degree firmware guard is not the operating endpoint). Passive linkage joints require measured/simulated states; URDF mimic does not represent these nonlinear closed loops.-->
   <!--PincOpen v1.0 derived meshes: Pollen Robotics, https://github.com/pollen-robotics/PincOpen/tree/v1.0, CC BY-SA 4.0 https://creativecommons.org/licenses/by-sa/4.0/ . Adaptations: rigid SO-101 attachment and CAD tessellation; derived PincOpen geometry remains CC BY-SA 4.0. XLeRobot RGBD gimbal: https://github.com/Vector-Wangel/XLeRobot/tree/137865981ca9e828d0923804cf77ededd22c7816 , Apache-2.0 https://www.apache.org/licenses/LICENSE-2.0 . Other geometry: supplied Cleany CAD and its retained component provenance.-->
   <xacro:macro name="cleany_robot_geometry" params="include_wheel_joints:=false">
@@ -1611,5 +1611,5 @@
       <origin xyz="0 -0.0490665820841 0" rpy="-1.57079632679 -0 -1.57079632679" />
       <axis xyz="0 0 -1" />
-      <limit lower="0" upper="1.0471975511965976" effort="1.5" velocity="4.245" />
+      <limit lower="0" upper="2.443460952792061" effort="1.5" velocity="4.245" />
     </joint>
     <link name="right_finger_1_internal">
@@ -1777,8 +1777,162 @@
         </material>
       </visual>
-      <collision name="right_finger_1_driving_collision_0">
-        <origin xyz="-1.29813049989e-05 -0.0162525771416 -0.00555" rpy="0 0 0" />
-        <geometry>
-          <box size="0.016120476541 0.0425051542832 0.0053000002" />
+      <collision name="right_finger_1_driving_collision_00">
+        <geometry>
+          <mesh filename="package://cleany_description/meshes/cad_v1/finger_1_driving_collision_00.stl" />
+        </geometry>
+      </collision>
+      <collision name="right_finger_1_driving_collision_01">
+        <geometry>
+          <mesh filename="package://cleany_description/meshes/cad_v1/finger_1_driving_collision_01.stl" />
+        </geometry>
+      </collision>
+      <collision name="right_finger_1_driving_collision_02">
+        <geometry>
+          <mesh filename="package://cleany_description/meshes/cad_v1/finger_1_driving_collision_02.stl" />
+        </geometry>
+      </collision>
+      <collision name="right_finger_1_driving_collision_03">
+        <geometry>
+          <mesh filename="package://cleany_description/meshes/cad_v1/finger_1_driving_collision_03.stl" />
+        </geometry>
+      </collision>
+      <collision name="right_finger_1_driving_collision_04">
+        <geometry>
+          <mesh filename="package://cleany_description/meshes/cad_v1/finger_1_driving_collision_04.stl" />
+        </geometry>
+      </collision>
+      <collision name="right_finger_1_driving_collision_05">
+        <geometry>
+          <mesh filename="package://cleany_description/meshes/cad_v1/finger_1_driving_collision_05.stl" />
+        </geometry>
+      </collision>
+      <collision name="right_finger_1_driving_collision_06">
+        <geometry>
+          <mesh filename="package://cleany_description/meshes/cad_v1/finger_1_driving_collision_06.stl" />
+        </geometry>
+      </collision>
+      <collision name="right_finger_1_driving_collision_07">
+        <geometry>
+          <mesh filename="package://cleany_description/meshes/cad_v1/finger_1_driving_collision_07.stl" />
+        </geometry>
+      </collision>
+      <collision name="right_finger_1_driving_collision_08">
+        <geometry>
+          <mesh filename="package://cleany_description/meshes/cad_v1/finger_1_driving_collision_08.stl" />
+        </geometry>
+      </collision>
+      <collision name="right_finger_1_driving_collision_09">
+        <geometry>
+          <mesh filename="package://cleany_description/meshes/cad_v1/finger_1_driving_collision_09.stl" />
+        </geometry>
+      </collision>
+      <collision name="right_finger_1_driving_collision_10">
+        <geometry>
+          <mesh filename="package://cleany_description/meshes/cad_v1/finger_1_driving_collision_10.stl" />
+        </geometry>
+      </collision>
+      <collision name="right_finger_1_driving_collision_11">
+        <geometry>
+          <mesh filename="package://cleany_description/meshes/cad_v1/finger_1_driving_collision_11.stl" />
+        </geometry>
+      </collision>
+      <collision name="right_finger_1_driving_collision_12">
+        <geometry>
+          <mesh filename="package://cleany_description/meshes/cad_v1/finger_1_driving_collision_12.stl" />
+        </geometry>
+      </collision>
+      <collision name="right_finger_1_driving_collision_13">
+        <geometry>
+          <mesh filename="package://cleany_description/meshes/cad_v1/finger_1_driving_collision_13.stl" />
+        </geometry>
+      </collision>
+      <collision name="right_finger_1_driving_collision_14">
+        <geometry>
+          <mesh filename="package://cleany_description/meshes/cad_v1/finger_1_driving_collision_14.stl" />
+        </geometry>
+      </collision>
+      <collision name="right_finger_1_driving_collision_15">
+        <geometry>
+          <mesh filename="package://cleany_description/meshes/cad_v1/finger_1_driving_collision_15.stl" />
+        </geometry>
+      </collision>
+      <collision name="right_finger_1_driving_collision_16">
+        <geometry>
+          <mesh filename="package://cleany_description/meshes/cad_v1/finger_1_driving_collision_16.stl" />
+        </geometry>
+      </collision>
+      <collision name="right_finger_1_driving_collision_17">
+        <geometry>
+          <mesh filename="package://cleany_description/meshes/cad_v1/finger_1_driving_collision_17.stl" />
+        </geometry>
+      </collision>
+      <collision name="right_finger_1_driving_collision_18">
+        <geometry>
+          <mesh filename="package://cleany_description/meshes/cad_v1/finger_1_driving_collision_18.stl" />
+        </geometry>
+      </collision>
+      <collision name="right_finger_1_driving_collision_19">
+        <geometry>
+          <mesh filename="package://cleany_description/meshes/cad_v1/finger_1_driving_collision_19.stl" />
+        </geometry>
+      </collision>
+      <collision name="right_finger_1_driving_collision_20">
+        <geometry>
+          <mesh filename="package://cleany_description/meshes/cad_v1/finger_1_driving_collision_20.stl" />
+        </geometry>
+      </collision>
+      <collision name="right_finger_1_driving_collision_21">
+        <geometry>
+          <mesh filename="package://cleany_description/meshes/cad_v1/finger_1_driving_collision_21.stl" />
+        </geometry>
+      </collision>
+      <collision name="right_finger_1_driving_collision_22">
+        <geometry>
+          <mesh filename="package://cleany_description/meshes/cad_v1/finger_1_driving_collision_22.stl" />
+        </geometry>
+      </collision>
+      <collision name="right_finger_1_driving_collision_23">
+        <geometry>
+          <mesh filename="package://cleany_description/meshes/cad_v1/finger_1_driving_collision_23.stl" />
+        </geometry>
+      </collision>
+      <collision name="right_finger_1_driving_collision_24">
+        <geometry>
+          <mesh filename="package://cleany_description/meshes/cad_v1/finger_1_driving_collision_24.stl" />
+        </geometry>
+      </collision>
+      <collision name="right_finger_1_driving_collision_25">
+        <geometry>
+          <mesh filename="package://cleany_description/meshes/cad_v1/finger_1_driving_collision_25.stl" />
+        </geometry>
+      </collision>
+      <collision name="right_finger_1_driving_collision_26">
+        <geometry>
+          <mesh filename="package://cleany_description/meshes/cad_v1/finger_1_driving_collision_26.stl" />
+        </geometry>
+      </collision>
+      <collision name="right_finger_1_driving_collision_27">
+        <geometry>
+          <mesh filename="package://cleany_description/meshes/cad_v1/finger_1_driving_collision_27.stl" />
+        </geometry>
+      </collision>
+      <collision name="right_finger_1_driving_collision_28">
+        <geometry>
+          <mesh filename="package://cleany_description/meshes/cad_v1/finger_1_driving_collision_28.stl" />
+        </geometry>
+      </collision>
+      <collision name="right_finger_1_driving_collision_29">
+        <geometry>
+          <mesh filename="package://cleany_description/meshes/cad_v1/finger_1_driving_collision_29.stl" />
+        </geometry>
+      </collision>
+      <collision name="right_finger_1_driving_collision_30">
+        <geometry>
+          <mesh filename="package://cleany_description/meshes/cad_v1/finger_1_driving_collision_30.stl" />
+        </geometry>
+      </collision>
+      <collision name="right_finger_1_driving_collision_31">
+        <geometry>
+          <mesh filename="package://cleany_description/meshes/cad_v1/finger_1_driving_collision_31.stl" />
         </geometry>
       </collision>
@@ -1961,8 +2115,162 @@
         </material>
       </visual>
-      <collision name="right_finger_2_driving_collision_0">
-        <origin xyz="-0.000514785589624 0.0162131654043 -0.00555" rpy="0 0 0" />
-        <geometry>
-          <box size="0.0165609229483 0.0424263308087 0.0053000002" />
+      <collision name="right_finger_2_driving_collision_00">
+        <geometry>
+          <mesh filename="package://cleany_description/meshes/cad_v1/finger_2_driving_collision_00.stl" />
+        </geometry>
+      </collision>
+      <collision name="right_finger_2_driving_collision_01">
+        <geometry>
+          <mesh filename="package://cleany_description/meshes/cad_v1/finger_2_driving_collision_01.stl" />
+        </geometry>
+      </collision>
+      <collision name="right_finger_2_driving_collision_02">
+        <geometry>
+          <mesh filename="package://cleany_description/meshes/cad_v1/finger_2_driving_collision_02.stl" />
+        </geometry>
+      </collision>
+      <collision name="right_finger_2_driving_collision_03">
+        <geometry>
+          <mesh filename="package://cleany_description/meshes/cad_v1/finger_2_driving_collision_03.stl" />
+        </geometry>
+      </collision>
+      <collision name="right_finger_2_driving_collision_04">
+        <geometry>
+          <mesh filename="package://cleany_description/meshes/cad_v1/finger_2_driving_collision_04.stl" />
+        </geometry>
+      </collision>
+      <collision name="right_finger_2_driving_collision_05">
+        <geometry>
+          <mesh filename="package://cleany_description/meshes/cad_v1/finger_2_driving_collision_05.stl" />
+        </geometry>
+      </collision>
+      <collision name="right_finger_2_driving_collision_06">
+        <geometry>
+          <mesh filename="package://cleany_description/meshes/cad_v1/finger_2_driving_collision_06.stl" />
+        </geometry>
+      </collision>
+      <collision name="right_finger_2_driving_collision_07">
+        <geometry>
+          <mesh filename="package://cleany_description/meshes/cad_v1/finger_2_driving_collision_07.stl" />
+        </geometry>
+      </collision>
+      <collision name="right_finger_2_driving_collision_08">
+        <geometry>
+          <mesh filename="package://cleany_description/meshes/cad_v1/finger_2_driving_collision_08.stl" />
+        </geometry>
+      </collision>
+      <collision name="right_finger_2_driving_collision_09">
+        <geometry>
+          <mesh filename="package://cleany_description/meshes/cad_v1/finger_2_driving_collision_09.stl" />
+        </geometry>
+      </collision>
+      <collision name="right_finger_2_driving_collision_10">
+        <geometry>
+          <mesh filename="package://cleany_description/meshes/cad_v1/finger_2_driving_collision_10.stl" />
+        </geometry>
+      </collision>
+      <collision name="right_finger_2_driving_collision_11">
+        <geometry>
+          <mesh filename="package://cleany_description/meshes/cad_v1/finger_2_driving_collision_11.stl" />
+        </geometry>
+      </collision>
+      <collision name="right_finger_2_driving_collision_12">
+        <geometry>
+          <mesh filename="package://cleany_description/meshes/cad_v1/finger_2_driving_collision_12.stl" />
+        </geometry>
+      </collision>
+      <collision name="right_finger_2_driving_collision_13">
+        <geometry>
+          <mesh filename="package://cleany_description/meshes/cad_v1/finger_2_driving_collision_13.stl" />
+        </geometry>
+      </collision>
+      <collision name="right_finger_2_driving_collision_14">
+        <geometry>
+          <mesh filename="package://cleany_description/meshes/cad_v1/finger_2_driving_collision_14.stl" />
+        </geometry>
+      </collision>
+      <collision name="right_finger_2_driving_collision_15">
+        <geometry>
+          <mesh filename="package://cleany_description/meshes/cad_v1/finger_2_driving_collision_15.stl" />
+        </geometry>
+      </collision>
+      <collision name="right_finger_2_driving_collision_16">
+        <geometry>
+          <mesh filename="package://cleany_description/meshes/cad_v1/finger_2_driving_collision_16.stl" />
+        </geometry>
+      </collision>
+      <collision name="right_finger_2_driving_collision_17">
+        <geometry>
+          <mesh filename="package://cleany_description/meshes/cad_v1/finger_2_driving_collision_17.stl" />
+        </geometry>
+      </collision>
+      <collision name="right_finger_2_driving_collision_18">
+        <geometry>
+          <mesh filename="package://cleany_description/meshes/cad_v1/finger_2_driving_collision_18.stl" />
+        </geometry>
+      </collision>
+      <collision name="right_finger_2_driving_collision_19">
+        <geometry>
+          <mesh filename="package://cleany_description/meshes/cad_v1/finger_2_driving_collision_19.stl" />
+        </geometry>
+      </collision>
+      <collision name="right_finger_2_driving_collision_20">
+        <geometry>
+          <mesh filename="package://cleany_description/meshes/cad_v1/finger_2_driving_collision_20.stl" />
+        </geometry>
+      </collision>
+      <collision name="right_finger_2_driving_collision_21">
+        <geometry>
+          <mesh filename="package://cleany_description/meshes/cad_v1/finger_2_driving_collision_21.stl" />
+        </geometry>
+      </collision>
+      <collision name="right_finger_2_driving_collision_22">
+        <geometry>
+          <mesh filename="package://cleany_description/meshes/cad_v1/finger_2_driving_collision_22.stl" />
+        </geometry>
+      </collision>
+      <collision name="right_finger_2_driving_collision_23">
+        <geometry>
+          <mesh filename="package://cleany_description/meshes/cad_v1/finger_2_driving_collision_23.stl" />
+        </geometry>
+      </collision>
+      <collision name="right_finger_2_driving_collision_24">
+        <geometry>
+          <mesh filename="package://cleany_description/meshes/cad_v1/finger_2_driving_collision_24.stl" />
+        </geometry>
+      </collision>
+      <collision name="right_finger_2_driving_collision_25">
+        <geometry>
+          <mesh filename="package://cleany_description/meshes/cad_v1/finger_2_driving_collision_25.stl" />
+        </geometry>
+      </collision>
+      <collision name="right_finger_2_driving_collision_26">
+        <geometry>
+          <mesh filename="package://cleany_description/meshes/cad_v1/finger_2_driving_collision_26.stl" />
+        </geometry>
+      </collision>
+      <collision name="right_finger_2_driving_collision_27">
+        <geometry>
+          <mesh filename="package://cleany_description/meshes/cad_v1/finger_2_driving_collision_27.stl" />
+        </geometry>
+      </collision>
+      <collision name="right_finger_2_driving_collision_28">
+        <geometry>
+          <mesh filename="package://cleany_description/meshes/cad_v1/finger_2_driving_collision_28.stl" />
+        </geometry>
+      </collision>
+      <collision name="right_finger_2_driving_collision_29">
+        <geometry>
+          <mesh filename="package://cleany_description/meshes/cad_v1/finger_2_driving_collision_29.stl" />
+        </geometry>
+      </collision>
+      <collision name="right_finger_2_driving_collision_30">
+        <geometry>
+          <mesh filename="package://cleany_description/meshes/cad_v1/finger_2_driving_collision_30.stl" />
+        </geometry>
+      </collision>
+      <collision name="right_finger_2_driving_collision_31">
+        <geometry>
+          <mesh filename="package://cleany_description/meshes/cad_v1/finger_2_driving_collision_31.stl" />
         </geometry>
       </collision>
@@ -2007,5 +2315,5 @@
       <origin xyz="0 -0.0490665820841 0" rpy="-1.57079632679 -0 -1.57079632679" />
       <axis xyz="0 0 -1" />
-      <limit lower="0" upper="1.0471975511965976" effort="1.5" velocity="4.245" />
+      <limit lower="0" upper="2.443460952792061" effort="1.5" velocity="4.245" />
     </joint>
     <link name="left_finger_1_internal">
@@ -2173,8 +2481,162 @@
         </material>
       </visual>
-      <collision name="left_finger_1_driving_collision_0">
-        <origin xyz="-1.29813049989e-05 -0.0162525771416 -0.00555" rpy="0 0 0" />
-        <geometry>
-          <box size="0.016120476541 0.0425051542832 0.0053000002" />
+      <collision name="left_finger_1_driving_collision_00">
+        <geometry>
+          <mesh filename="package://cleany_description/meshes/cad_v1/finger_1_driving_collision_00.stl" />
+        </geometry>
+      </collision>
+      <collision name="left_finger_1_driving_collision_01">
+        <geometry>
+          <mesh filename="package://cleany_description/meshes/cad_v1/finger_1_driving_collision_01.stl" />
+        </geometry>
+      </collision>
+      <collision name="left_finger_1_driving_collision_02">
+        <geometry>
+          <mesh filename="package://cleany_description/meshes/cad_v1/finger_1_driving_collision_02.stl" />
+        </geometry>
+      </collision>
+      <collision name="left_finger_1_driving_collision_03">
+        <geometry>
+          <mesh filename="package://cleany_description/meshes/cad_v1/finger_1_driving_collision_03.stl" />
+        </geometry>
+      </collision>
+      <collision name="left_finger_1_driving_collision_04">
+        <geometry>
+          <mesh filename="package://cleany_description/meshes/cad_v1/finger_1_driving_collision_04.stl" />
+        </geometry>
+      </collision>
+      <collision name="left_finger_1_driving_collision_05">
+        <geometry>
+          <mesh filename="package://cleany_description/meshes/cad_v1/finger_1_driving_collision_05.stl" />
+        </geometry>
+      </collision>
+      <collision name="left_finger_1_driving_collision_06">
+        <geometry>
+          <mesh filename="package://cleany_description/meshes/cad_v1/finger_1_driving_collision_06.stl" />
+        </geometry>
+      </collision>
+      <collision name="left_finger_1_driving_collision_07">
+        <geometry>
+          <mesh filename="package://cleany_description/meshes/cad_v1/finger_1_driving_collision_07.stl" />
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