Commit message: fix(model): restore 140 degree PincOpen travel with fitted rod collisions

File: ros2_ws/src/cleany_description/urdf/head_camera.xacro (robot description, xacro)
@@ -173,5 +173,5 @@
    limitations under the License.
 -->
-  <!--CAD source Cleany.FCStd SHA256 5fe6b78e2eb0ef183e66631eb8aef31503eb8f0b0c5902d9955affd8a7aef82e. Export units: metres and radians; visual tessellation 0.12 mm. Saved CAD folded pose is cad_home in cad_v1.xml. Public left/right follows REP-103 base +Y/-Y; CAD internal RightArm is ROS left. Positive gripper angle opens: 0 to pi/3 corresponds to source cam 0 to -60 degrees. Passive linkage joints require measured/simulated states; URDF mimic does not represent these nonlinear closed loops.-->
+  <!--CAD source Cleany.FCStd SHA256 5fe6b78e2eb0ef183e66631eb8aef31503eb8f0b0c5902d9955affd8a7aef82e. Export units: metres and radians; visual tessellation 0.12 mm. Saved CAD folded pose is cad_home in cad_v1.xml. Public left/right follows REP-103 base +Y/-Y; CAD internal RightArm is ROS left. Positive gripper angle opens: 0 to 2.443460952792061 radians corresponds to source cam 0 to -140 degrees (vendor v1.0 flash_test.ipynb open command; 147-degree firmware guard is not the operating endpoint). Passive linkage joints require measured/simulated states; URDF mimic does not represent these nonlinear closed loops.-->
   <!--PincOpen v1.0 derived meshes: Pollen Robotics, https://github.com/pollen-robotics/PincOpen/tree/v1.0, CC BY-SA 4.0 https://creativecommons.org/licenses/by-sa/4.0/ . Adaptations: rigid SO-101 attachment and CAD tessellation; derived PincOpen geometry remains CC BY-SA 4.0. XLeRobot RGBD gimbal: https://github.com/Vector-Wangel/XLeRobot/tree/137865981ca9e828d0923804cf77ededd22c7816 , Apache-2.0 https://www.apache.org/licenses/LICENSE-2.0 . Other geometry: supplied Cleany CAD and its retained component provenance.-->
   <xacro:macro name="cleany_head_camera">
