Commit message: feat(description): reflect physical head mount and calibrated camera frames

File: ros2_ws/src/cleany_description/urdf/cleany.urdf.xacro (robot description, xacro)
@@ -1,4 +1,6 @@
 <?xml version="1.0"?>
 <robot name="cleany" xmlns:xacro="http://www.ros.org/wiki/xacro">
+  <xacro:arg name="head_mast_rear_gap_m" default="0.05"/>
+  <xacro:arg name="calibration_profile" default=""/>
   <xacro:arg name="include_head_camera" default="true"/>
   <xacro:arg name="include_wheel_joints" default="true"/>
@@ -6,7 +8,18 @@
   <xacro:include filename="$(find cleany_description)/urdf/cleany_geometry.xacro"/>
   <xacro:include filename="$(find cleany_description)/urdf/head_camera.xacro"/>
-  <xacro:cleany_robot_geometry include_wheel_joints="$(arg include_wheel_joints)"/>
+  <xacro:include filename="$(find cleany_description)/urdf/camera_calibration.xacro"/>
+  <xacro:property name="calibration_directory"
+                  value="$(find cleany_description)/config/calibration/$(arg calibration_profile)"/>
+  <xacro:cleany_robot_geometry include_wheel_joints="$(arg include_wheel_joints)"
+                              head_mast_rear_gap_m="$(arg head_mast_rear_gap_m)"/>
+  <xacro:if value="${'$(arg calibration_profile)' != ''}">
+    <xacro:cleany_calibrated_wrist_camera side="left"
+      calibration_file="${calibration_directory + '/left_wrist_camera_extrinsics.yaml'}"/>
+    <xacro:cleany_calibrated_wrist_camera side="right"
+      calibration_file="${calibration_directory + '/right_wrist_camera_extrinsics.yaml'}"/>
+  </xacro:if>
   <xacro:if value="$(arg include_head_camera)">
-    <xacro:cleany_head_camera/>
+    <xacro:cleany_head_camera
+      calibration_file="${calibration_directory + '/head_rgb_extrinsics.yaml' if '$(arg calibration_profile)' != '' else ''}"/>
   </xacro:if>
 </robot>

File: ros2_ws/src/cleany_description/urdf/cleany_control.urdf.xacro (robot description, xacro)
@@ -3,4 +3,5 @@
   <xacro:arg name="mujoco_model" default=""/>
   <xacro:arg name="mujoco_hardware_plugin" default="mujoco_ros2_control/MujocoSystemInterface"/>
+  <xacro:arg name="head_mast_rear_gap_m" default="0.05"/>
   <xacro:arg name="headless" default="true"/>
   <xacro:arg name="sim_speed_factor" default="1.0"/>
@@ -26,5 +27,5 @@
   <xacro:include filename="$(find cleany_description)/urdf/cleany_geometry.xacro"/>
   <xacro:include filename="$(find cleany_description)/urdf/cleany_mujoco_ros2_control.xacro"/>
-  <xacro:cleany_robot_geometry/>
+  <xacro:cleany_robot_geometry head_mast_rear_gap_m="$(arg head_mast_rear_gap_m)"/>
   <xacro:cleany_mujoco_ros2_control
     mujoco_model="$(arg mujoco_model)"

File: ros2_ws/src/cleany_description/urdf/cleany_geometry.xacro (robot description, xacro)
@@ -3,7 +3,7 @@
   <xacro:include filename="$(find cleany_description)/urdf/dual_arm.xacro" />
   <xacro:include filename="$(find cleany_description)/urdf/head_camera.xacro" />
-  <xacro:macro name="cleany_robot_geometry" params="include_wheel_joints:=false">
+  <xacro:macro name="cleany_robot_geometry" params="include_wheel_joints:=false head_mast_rear_gap_m:=0.05">
     <!-- Fixed mast belongs to every model, including the controller's TF tree. -->
-    <xacro:cleany_head_mount/>
+    <xacro:cleany_head_mount rear_gap_m="${head_mast_rear_gap_m}"/>
     <link name="base_link">
       <xacro:cleany_link_properties link_name="base_link" />

File: ros2_ws/src/cleany_description/urdf/dual_arm.xacro (robot description, xacro)
@@ -77,6 +77,6 @@
       <origin xyz="0 -0.140 0" rpy="0 0 0" />
     </joint>
-    <!-- Wrist camera extrinsics are evaluation-only until calibrated.
-         Do not publish the MJCF ground-truth optical edge into runtime TF. -->
+    <!-- Measured wrist optical frames are added by the optional calibration profile.
+         MJCF ground-truth camera frames remain separate from runtime TF. -->
   </xacro:macro>
 </robot>

File: ros2_ws/src/cleany_description/urdf/head_camera.xacro (robot description, xacro)
@@ -1,4 +1,10 @@
 <robot xmlns:xacro="http://www.ros.org/wiki/xacro">
-  <xacro:macro name="cleany_head_mount">
+  <xacro:macro name="cleany_head_mount" params="rear_gap_m:=0.05">
+    <!-- 2026-10-09 assembly: smooth mast face points rearward and sits
+         rear_gap_m behind the CAD top plate's rear edge (base_link -X).
+         Plate: center X=0.1162, depth=0.16. Mast smooth face: local X=-0.131.
+         Rotate the rigid mast by pi relative to the previous assembly. -->
+    <xacro:property name="plate_rear_x_m" value="${0.1162 - 0.16 / 2.0}"/>
+    <xacro:property name="mast_smooth_face_x_m" value="${-0.131}"/>
     <link name="top_base_link">
       <xacro:cleany_link_properties link_name="top_base_link" />
@@ -7,8 +13,10 @@
       <parent link="base_link" />
       <child link="top_base_link" />
-      <origin xyz="0 0 0.35" rpy="0 0 3.14159265359" />
+      <origin xyz="${plate_rear_x_m - float(rear_gap_m) - mast_smooth_face_x_m} 0 0.35" rpy="0 0 0" />
     </joint>
   </xacro:macro>
-  <xacro:macro name="cleany_head_camera">
+  <xacro:macro name="cleany_head_camera" params="calibration_file:=''">
+    <xacro:property name="rgb_calibration"
+      value="${xacro.load_yaml(calibration_file) if calibration_file else dict(xyz='0 0 0', rpy='-1.57079632679 0 -1.57079632679')}"/>
     <link name="head_pan_link">
       <xacro:cleany_link_properties link_name="head_pan_link" />
@@ -17,5 +25,6 @@
       <parent link="top_base_link" />
       <child link="head_pan_link" />
-      <origin xyz="-0.103 0 0.323" rpy="0 0 0" />
+      <!-- Reversed mast; 65 mm lower mount + 238 mm pillar. -->
+      <origin xyz="-0.103 0 0.3505" rpy="0 0 ${pi}" />
       <axis xyz="0 0 1" />
       <limit lower="-3.2" upper="3.2" effort="2.6477955" velocity="4.245" />
@@ -53,5 +62,5 @@
       <parent link="head_camera_rgb_frame" />
       <child link="head_camera_rgb_optical_frame" />
-      <origin xyz="0 0 0" rpy="-1.57079632679 0 -1.57079632679" />
+      <origin xyz="${rgb_calibration['xyz']}" rpy="${rgb_calibration['rpy']}" />
     </joint>
     <link name="head_camera_depth_frame">

File: ros2_ws/src/cleany_description/urdf/physical_properties.xacro (robot description, xacro)
@@ -1046,5 +1046,5 @@
       </visual>
       <visual name="mjcf_geom_113_0_visual">
-        <origin xyz="-0.297999984077 0.00600079076974 -0.715" rpy="-5.90619133461e-17 6.93889390391e-18 3.13999734641" />
+        <origin xyz="-0.297999984077 0.00600079076974 -0.6875" rpy="-5.90619133461e-17 6.93889390391e-18 3.13999734641" />
         <geometry>
           <mesh filename="package://cleany_description/meshes/topbase2.stl" scale="0.001 0.001 0.001" />
@@ -1055,7 +1055,14 @@
       </visual>
       <collision name="mjcf_geom_114_0_collision">
-        <origin xyz="-0.1044 -0.00025 0.23595" rpy="0 -0 5.25245130592e-18" />
-        <geometry>
-          <box size="0.1504 0.12 0.3349" />
+        <origin xyz="-0.1044 -0.00025 0.2822" rpy="0 -0 5.25245130592e-18" />
+        <geometry>
+          <box size="0.1504 0.12 0.2974" />
+        </geometry>
+      </collision>
+      <collision name="lower_head_mount_collision">
+        <!-- 172 mm depth; front edge 41 mm behind the top plate's front edge. -->
+        <origin xyz="-0.048 -0.00025 0.101" rpy="0 0 0" />
+        <geometry>
+          <box size="0.172 0.12 0.065" />
         </geometry>
       </collision>
