Commit message: fix(description): stabilize base inertia parity across MuJoCo versions

File: ros2_ws/src/cleany_description/urdf/physical_properties.xacro (robot description, xacro)
@@ -2,9 +2,9 @@
   <xacro:macro name="cleany_link_properties" params="link_name">
     <xacro:if value="${link_name == 'base_link'}">
-      <!-- Combined chassis and fixed arm-base inertia at the aligned mounts. -->
+      <!-- Combined source MJCF fullinertia tensors at the aligned arm mounts. -->
       <inertial>
         <origin xyz="0.00644073126036 2.68998835469e-05 -0.141372186369" rpy="0 -0 0" />
         <mass value="12.3513377764" />
-        <inertia ixx="0.933542754865" ixy="0.000607852427179" ixz="-0.0463142424415" iyy="0.865629751875" iyz="-4.37794203494e-08" izz="0.487782920537" />
+        <inertia ixx="0.933542754865" ixy="0.000607854672282" ixz="-0.0463142424415" iyy="0.865629751875" iyz="-1.47964742646e-08" izz="0.487782920537" />
       </inertial>
       <visual name="mjcf_geom_0_0_visual">

Commit message: feat(description): apply Jetson v8 wrist camera mounts

File: ros2_ws/src/cleany_description/urdf/physical_properties.xacro (robot description, xacro)
@@ -1,3 +1,4 @@
 <robot xmlns:xacro="http://www.ros.org/wiki/xacro">
+  <xacro:include filename="wrist_mount_v8.xacro" />
   <xacro:macro name="cleany_link_properties" params="link_name">
     <xacro:if value="${link_name == 'base_link'}">
@@ -650,34 +651,5 @@
         </geometry>
       </collision>
-      <visual name="mjcf_geom_78_0_visual">
-        <origin xyz="5.51022591132e-08 -0.00699996818156 0.0239988737994" rpy="1.57079632677 6.32679579342e-06 -1.57079999999" />
-        <geometry>
-          <mesh filename="package://cleany_description/meshes/XLeRobot_camera1.stl" scale="0.001 0.001 0.001" />
-        </geometry>
-        <material name="mjcf_color_78">
-          <color rgba="0.300000011921 0.300000011921 0.300000011921 1" />
-        </material>
-      </visual>
-      <collision name="mjcf_geom_78_0_self_filter_collision">
-        <origin xyz="5.51022591132e-08 -0.00699996818156 0.0239988737994" rpy="1.57079632677 6.32679579342e-06 -1.57079999999" />
-        <geometry>
-          <mesh filename="package://cleany_description/meshes/XLeRobot_camera1.stl" scale="0.001 0.001 0.001" />
-        </geometry>
-      </collision>
-      <visual name="mjcf_geom_79_0_visual">
-        <origin xyz="5.51022591513e-08 -0.00699996818156 0.0239988737994" rpy="1.57079632677 6.3267957937e-06 -1.57079999999" />
-        <geometry>
-          <mesh filename="package://cleany_description/meshes/XLeRobot_camera2.stl" scale="0.001 0.001 0.001" />
-        </geometry>
-        <material name="mjcf_color_79">
-          <color rgba="0.10000000149 0.10000000149 0.10000000149 1" />
-        </material>
-      </visual>
-      <collision name="mjcf_geom_79_0_self_filter_collision">
-        <origin xyz="5.51022591513e-08 -0.00699996818156 0.0239988737994" rpy="1.57079632677 6.3267957937e-06 -1.57079999999" />
-        <geometry>
-          <mesh filename="package://cleany_description/meshes/XLeRobot_camera2.stl" scale="0.001 0.001 0.001" />
-        </geometry>
-      </collision>
+      <xacro:cleany_wrist_mount_v8 side="left" />
     </xacro:if>
     <xacro:if value="${link_name == 'left_moving_jaw_link'}">
@@ -944,34 +916,5 @@
         </geometry>
       </collision>
-      <visual name="mjcf_geom_110_0_visual">
-        <origin xyz="5.50979259921e-08 -0.00599990458298 0.0240000535035" rpy="1.57079632678 3.676795793e-06 -1.5708" />
-        <geometry>
-          <mesh filename="package://cleany_description/meshes/XLeRobot_camera1.stl" scale="0.001 0.001 0.001" />
-        </geometry>
-        <material name="mjcf_color_110">
-          <color rgba="0.300000011921 0.300000011921 0.300000011921 1" />
-        </material>
-      </visual>
-      <collision name="mjcf_geom_110_0_self_filter_collision">
-        <origin xyz="5.50979259921e-08 -0.00599990458298 0.0240000535035" rpy="1.57079632678 3.676795793e-06 -1.5708" />
-        <geometry>
-          <mesh filename="package://cleany_description/meshes/XLeRobot_camera1.stl" scale="0.001 0.001 0.001" />
-        </geometry>
-      </collision>
-      <visual name="mjcf_geom_111_0_visual">
-        <origin xyz="5.50979259431e-08 -0.00599990458298 0.0240000535035" rpy="1.57079632678 3.67679579317e-06 -1.5708" />
-        <geometry>
-          <mesh filename="package://cleany_description/meshes/XLeRobot_camera2.stl" scale="0.001 0.001 0.001" />
-        </geometry>
-        <material name="mjcf_color_111">
-          <color rgba="0.10000000149 0.10000000149 0.10000000149 1" />
-        </material>
-      </visual>
-      <collision name="mjcf_geom_111_0_self_filter_collision">
-        <origin xyz="5.50979259431e-08 -0.00599990458298 0.0240000535035" rpy="1.57079632678 3.67679579317e-06 -1.5708" />
-        <geometry>
-          <mesh filename="package://cleany_description/meshes/XLeRobot_camera2.stl" scale="0.001 0.001 0.001" />
-        </geometry>
-      </collision>
+      <xacro:cleany_wrist_mount_v8 side="right" />
     </xacro:if>
     <xacro:if value="${link_name == 'right_moving_jaw_link'}">

Commit message: feat(jetson): curate physical manipulation integration on main

File: ros2_ws/src/cleany_description/urdf/physical_properties.xacro (robot description, xacro)
@@ -1,4 +1,9 @@
 <robot xmlns:xacro="http://www.ros.org/wiki/xacro">
   <xacro:include filename="wrist_mount_v8.xacro" />
+  <!-- Physical collection can use the validated head CAD collision surfaces. -->
+  <xacro:arg name="head_collision_meshes" default="false"/>
+  <!-- Separate enclosing arm collision assets; visual CAD and inertia stay exact. -->
+  <xacro:arg name="optimized_arm_collision_meshes" default="false"/>
+  <xacro:property name="arm_collision_directory" value="${'collision/' if '$(arg optimized_arm_collision_meshes)'.lower() in ('true', '1') else ''}"/>
   <xacro:macro name="cleany_link_properties" params="link_name">
     <xacro:if value="${link_name == 'base_link'}">
@@ -403,5 +408,5 @@
         <origin xyz="0.116200343 0.151031727 0.431297" rpy="0 -0 3.14159265359" />
         <geometry>
-          <mesh filename="package://cleany_description/meshes/Base.stl" scale="1 1 1" />
+          <mesh filename="package://cleany_description/meshes/${arm_collision_directory}Base.stl" scale="1 1 1" />
         </geometry>
       </collision>
@@ -409,5 +414,5 @@
         <origin xyz="0.116200343 0.151031727 0.431297" rpy="0 -0 3.14159265359" />
         <geometry>
-          <mesh filename="package://cleany_description/meshes/Base_Motor.stl" scale="1 1 1" />
+          <mesh filename="package://cleany_description/meshes/${arm_collision_directory}Base_Motor.stl" scale="1 1 1" />
         </geometry>
       </collision>
@@ -433,5 +438,5 @@
         <origin xyz="0.116200838 -0.150977072 0.431297" rpy="0 -5.55111512313e-17 -3.58979312866e-09" />
         <geometry>
-          <mesh filename="package://cleany_description/meshes/Base.stl" scale="1 1 1" />
+          <mesh filename="package://cleany_description/meshes/${arm_collision_directory}Base.stl" scale="1 1 1" />
         </geometry>
       </collision>
@@ -439,5 +444,5 @@
         <origin xyz="0.116200838 -0.150977072 0.431297" rpy="0 -0 -3.58979302984e-09" />
         <geometry>
-          <mesh filename="package://cleany_description/meshes/Base_Motor.stl" scale="1 1 1" />
+          <mesh filename="package://cleany_description/meshes/${arm_collision_directory}Base_Motor.stl" scale="1 1 1" />
         </geometry>
       </collision>
@@ -476,5 +481,5 @@
         <origin xyz="6.93889390391e-18 -9.71445146547e-17 6.24500451352e-17" rpy="-3.35618590807e-13 -2.65358979329e-06 9.74722386141e-12" />
         <geometry>
-          <mesh filename="package://cleany_description/meshes/Rotation_Pitch_Motor.stl" scale="1 1 1" />
+          <mesh filename="package://cleany_description/meshes/${arm_collision_directory}Rotation_Pitch_Motor.stl" scale="1 1 1" />
         </geometry>
       </collision>
@@ -516,5 +521,5 @@
         <origin xyz="-0.000100253949776 0.0650999997343 -0.0120000000001" rpy="1.57079632678 -6.71128083662e-13 -1.57079367321" />
         <geometry>
-          <mesh filename="package://cleany_description/meshes/Upper_Arm_5cm.stl" scale="1 1 1" />
+          <mesh filename="package://cleany_description/meshes/${arm_collision_directory}Upper_Arm_5cm.stl" scale="1 1 1" />
         </geometry>
       </collision>
@@ -522,5 +527,5 @@
         <origin xyz="-2.13880336414e-07 0.0499999999997 -4.37740121928e-14" rpy="-6.70963993052e-13 1.94943609866e-11 2.65358979315e-06" />
         <geometry>
-          <mesh filename="package://cleany_description/meshes/Upper_Arm_Motor.stl" scale="1 1 1" />
+          <mesh filename="package://cleany_description/meshes/${arm_collision_directory}Upper_Arm_Motor.stl" scale="1 1 1" />
         </geometry>
       </collision>
@@ -562,5 +567,5 @@
         <origin xyz="-0.00250068507803 0.0320000000001 0.0649999933651" rpy="-1.26408588281e-07 1.57079367321 -1.26413818102e-07" />
         <geometry>
-          <mesh filename="package://cleany_description/meshes/Lower_Arm_5cm.stl" scale="1 1 1" />
+          <mesh filename="package://cleany_description/meshes/${arm_collision_directory}Lower_Arm_5cm.stl" scale="1 1 1" />
         </geometry>
       </collision>
@@ -605,5 +610,5 @@
         <origin xyz="-1.0032431971e-06 1.34827565779e-12 1.81325612443e-13" rpy="1.71455341476e-18 9.38558131561e-18 -2.65358979335e-06" />
         <geometry>
-          <mesh filename="package://cleany_description/meshes/Wrist_Pitch_Roll_Motor.stl" scale="1 1 1" />
+          <mesh filename="package://cleany_description/meshes/${arm_collision_directory}Wrist_Pitch_Roll_Motor.stl" scale="1 1 1" />
         </geometry>
       </collision>
@@ -636,5 +641,5 @@
         <origin xyz="4.08954814457e-12 1.5600333525e-12 -1.16272394365e-06" rpy="2.65358979332e-06 -3.35582256428e-13 9.74717818498e-12" />
         <geometry>
-          <mesh filename="package://cleany_description/meshes/Fixed_Jaw_Motor.stl" scale="1 1 1" />
+          <mesh filename="package://cleany_description/meshes/${arm_collision_directory}Fixed_Jaw_Motor.stl" scale="1 1 1" />
         </geometry>
       </collision>
@@ -741,5 +746,5 @@
         <origin xyz="-2.58639897693e-13 -1.2490009027e-16 -1.04083408559e-17" rpy="-3.35608339132e-13 -3.58979290442e-09 1.32290012278e-14" />
         <geometry>
-          <mesh filename="package://cleany_description/meshes/Rotation_Pitch_Motor.stl" scale="1 1 1" />
+          <mesh filename="package://cleany_description/meshes/${arm_collision_directory}Rotation_Pitch_Motor.stl" scale="1 1 1" />
         </geometry>
       </collision>
@@ -781,5 +786,5 @@
         <origin xyz="-0.000100000343803 0.0650999999996 -0.0120000000001" rpy="1.57079632679 -6.71155839238e-13 -1.57079632321" />
         <geometry>
-          <mesh filename="package://cleany_description/meshes/Upper_Arm_5cm.stl" scale="1 1 1" />
+          <mesh filename="package://cleany_description/meshes/${arm_collision_directory}Upper_Arm_5cm.stl" scale="1 1 1" />
         </geometry>
       </collision>
@@ -787,5 +792,5 @@
         <origin xyz="-2.89597327455e-10 0.05 -4.3832992791e-14" rpy="-6.70993330038e-13 2.63712662818e-14 3.589792896e-09" />
         <geometry>
-          <mesh filename="package://cleany_description/meshes/Upper_Arm_Motor.stl" scale="1 1 1" />
+          <mesh filename="package://cleany_description/meshes/${arm_collision_directory}Upper_Arm_Motor.stl" scale="1 1 1" />
         </geometry>
       </collision>
@@ -827,5 +832,5 @@
         <origin xyz="-0.00250000092704 0.0320000000001 0.064999999991" rpy="0 1.57079632321 1.31376029847e-14" />
         <geometry>
-          <mesh filename="package://cleany_description/meshes/Lower_Arm_5cm.stl" scale="1 1 1" />
+          <mesh filename="package://cleany_description/meshes/${arm_collision_directory}Lower_Arm_5cm.stl" scale="1 1 1" />
         </geometry>
       </collision>
@@ -870,5 +875,5 @@
         <origin xyz="-1.35745236753e-09 1.73819292293e-14 1.81325653127e-13" rpy="-4.23516473627e-22 -1.52033649196e-30 -3.5897930184e-09" />
         <geometry>
-          <mesh filename="package://cleany_description/meshes/Wrist_Pitch_Roll_Motor.stl" scale="1 1 1" />
+          <mesh filename="package://cleany_description/meshes/${arm_collision_directory}Wrist_Pitch_Roll_Motor.stl" scale="1 1 1" />
         </geometry>
       </collision>
@@ -901,5 +906,5 @@
         <origin xyz="-1.75451667084e-13 1.72466207982e-14 -1.57319893348e-09" rpy="3.58979298692e-09 -3.3556837864e-13 1.31342831277e-14" />
         <geometry>
-          <mesh filename="package://cleany_description/meshes/Fixed_Jaw_Motor.stl" scale="1 1 1" />
+          <mesh filename="package://cleany_description/meshes/${arm_collision_directory}Fixed_Jaw_Motor.stl" scale="1 1 1" />
         </geometry>
       </collision>
@@ -997,5 +1002,17 @@
         </material>
       </visual>
+      <xacro:if value="$(arg head_collision_meshes)">
+        <collision name="head_mast_cad_collision">
+          <origin xyz="-0.440000013266 -0.00499883242047 -0.6" rpy="-1.73472347598e-18 6.93889390391e-18 -2.65358979331e-06" />
+          <geometry><mesh filename="package://cleany_description/meshes/cad_frame/topbase1.stl" scale="1 1 1" /></geometry>
+        </collision>
+        <collision name="lower_head_mount_cad_collision">
+          <origin xyz="-0.297999984077 0.00600079076974 -0.6875" rpy="-5.90619133461e-17 6.93889390391e-18 3.13999734641" />
+          <geometry><mesh filename="package://cleany_description/meshes/topbase2.stl" scale="0.001 0.001 0.001" /></geometry>
+        </collision>
+      </xacro:if>
+      <xacro:unless value="$(arg head_collision_meshes)">
       <collision name="mjcf_geom_114_0_collision">
+        <!-- Retain pillar coverage above the independently positioned lower mount. -->
         <origin xyz="-0.1044 -0.00025 0.2822" rpy="0 -0 5.25245130592e-18" />
         <geometry>
@@ -1010,4 +1027,5 @@
         </geometry>
       </collision>
+      </xacro:unless>
     </xacro:if>
     <xacro:if value="${link_name == 'head_pan_link'}">
@@ -1035,4 +1053,15 @@
         </material>
       </visual>
+      <xacro:if value="$(arg head_collision_meshes)">
+        <collision name="head_pan_bracket_cad_collision">
+          <origin xyz="-0.335000013266 -0.00499883772765 -0.923" rpy="8.67361737988e-19 -5.55111512313e-17 -2.65358979336e-06" />
+          <geometry><mesh filename="package://cleany_description/meshes/tophead1.stl" scale="0.001 0.001 0.001" /></geometry>
+        </collision>
+        <collision name="head_pan_motor_cad_collision">
+          <origin xyz="1.16999997611 -0.00900283138028 0.262" rpy="-3.14159201945 -1.57000000101 3.14159063414" />
+          <geometry><mesh filename="package://cleany_description/meshes/tophead4.stl" scale="0.001 0.001 0.001" /></geometry>
+        </collision>
+      </xacro:if>
+      <xacro:unless value="$(arg head_collision_meshes)">
       <collision name="mjcf_geom_117_0_collision">
         <origin xyz="0.0135 1.09426068873e-19 0.093" rpy="0 -0 5.25245130592e-18" />
@@ -1041,4 +1070,5 @@
         </geometry>
       </collision>
+      </xacro:unless>
     </xacro:if>
     <xacro:if value="${link_name == 'head_tilt_link'}">
@@ -1066,4 +1096,15 @@
         </material>
       </visual>
+      <xacro:if value="$(arg head_collision_meshes)">
+        <collision name="head_tilt_bracket_cad_collision">
+          <origin xyz="0.162649962825 -0.00600113446269 -1.16815" rpy="-6.20163642662e-17 4.55026099265e-18 -5.31076937972e-06" />
+          <geometry><mesh filename="package://cleany_description/meshes/tophead5.stl" scale="0.001 0.001 0.001" /></geometry>
+        </collision>
+        <collision name="head_tilt_motor_cad_collision">
+          <origin xyz="0.162649962825 -0.00600113446269 -1.16815" rpy="-3.56491214576e-17 -1.75849280414e-18 -5.31076937974e-06" />
+          <geometry><mesh filename="package://cleany_description/meshes/tophead6.stl" scale="0.001 0.001 0.001" /></geometry>
+        </collision>
+      </xacro:if>
+      <xacro:unless value="$(arg head_collision_meshes)">
       <collision name="mjcf_geom_120_0_collision">
         <origin xyz="0.0101 0.0026 0.014" rpy="0 -0 7.23196730366e-18" />
@@ -1072,4 +1113,5 @@
         </geometry>
       </collision>
+      </xacro:unless>
     </xacro:if>
     <xacro:if value="${link_name == 'front_right_wheel_link'}">

File: ros2_ws/src/cleany_moveit_config/config/cleany_mock.urdf.xacro (robot description, xacro)
@@ -1,13 +1,19 @@
 <?xml version="1.0"?>
 <robot name="cleany" xmlns:xacro="http://www.ros.org/wiki/xacro">
+  <xacro:arg name="include_head_camera" default="false"/>
+  <xacro:arg name="head_tilt_initial" default="0.405"/>
   <!-- Reuse the canonical geometry; this file only adds a mock ros2_control system. -->
   <xacro:include filename="$(find cleany_description)/urdf/materials.xacro"/>
   <xacro:include filename="$(find cleany_description)/urdf/cleany_geometry.xacro"/>
+  <xacro:include filename="$(find cleany_description)/urdf/head_camera.xacro"/>
   <xacro:cleany_robot_geometry/>
-  <xacro:macro name="cleany_mock_joint" params="joint_name">
+  <xacro:if value="$(arg include_head_camera)">
+    <xacro:cleany_head_camera mount_x_offset_m="-0.10"/>
+  </xacro:if>
+  <xacro:macro name="cleany_mock_joint" params="joint_name initial_value:=0.0">
     <joint name="${joint_name}">
       <command_interface name="position"/>
       <state_interface name="position">
-        <param name="initial_value">0.0</param>
+        <param name="initial_value">${initial_value}</param>
       </state_interface>
       <state_interface name="velocity"/>
@@ -30,4 +36,8 @@
     <xacro:cleany_mock_joint joint_name="right_wrist_roll_joint"/>
     <xacro:cleany_mock_joint joint_name="right_gripper_joint"/>
+    <xacro:if value="$(arg include_head_camera)">
+      <xacro:cleany_mock_joint joint_name="head_pan_joint" initial_value="0.023"/>
+      <xacro:cleany_mock_joint joint_name="head_tilt_joint" initial_value="$(arg head_tilt_initial)"/>
+    </xacro:if>
   </ros2_control>
 </robot>
