Commit message: chore: checkpoint Jetson integration work before main sync
Preserve semantic label contracts, manipulation updates, collision geometry, monitor UI, validation tools, and implementation documentation. Record the current KB submodule revision; keep local output artifacts outside Git.

File: ros2_ws/src/cleany_description/urdf/physical_properties.xacro (robot description, xacro)
@@ -475,5 +475,5 @@
         <origin xyz="-2.98155597434e-19 -9.71445146547e-17 5.55111512313e-17" rpy="-3.3539837574e-13 -2.65358979332e-06 9.74718396277e-12" />
         <geometry>
-          <mesh filename="package://cleany_description/meshes/Rotation_Pitch.stl" scale="1 1 1" />
+          <mesh filename="package://cleany_description/meshes/${arm_collision_directory}Rotation_Pitch.stl" scale="1 1 1" />
         </geometry>
       </collision>
@@ -573,5 +573,5 @@
         <origin xyz="-6.45273883274e-07 1.36086454605e-13 0.0499999999991" rpy="-3.35508353651e-13 -2.65358979335e-06 9.74729819568e-12" />
         <geometry>
-          <mesh filename="package://cleany_description/meshes/Lower_Arm_Motor.stl" scale="1 1 1" />
+          <mesh filename="package://cleany_description/meshes/${arm_collision_directory}Lower_Arm_Motor.stl" scale="1 1 1" />
         </geometry>
       </collision>
@@ -604,5 +604,5 @@
         <origin xyz="-1.00324319708e-06 1.34834851617e-12 1.81327947991e-13" rpy="-1.19262238973e-17 7.3725747729e-18 -2.65358979346e-06" />
         <geometry>
-          <mesh filename="package://cleany_description/meshes/Wrist_Pitch_Roll.stl" scale="1 1 1" />
+          <mesh filename="package://cleany_description/meshes/${arm_collision_directory}Wrist_Pitch_Roll.stl" scale="1 1 1" />
         </geometry>
       </collision>
@@ -740,5 +740,5 @@
         <origin xyz="-2.58642499779e-13 -1.5959455979e-16 -4.51028103754e-17" rpy="-3.3545388689e-13 -3.5897930236e-09 1.31917046731e-14" />
         <geometry>
-          <mesh filename="package://cleany_description/meshes/Rotation_Pitch.stl" scale="1 1 1" />
+          <mesh filename="package://cleany_description/meshes/${arm_collision_directory}Rotation_Pitch.stl" scale="1 1 1" />
         </geometry>
       </collision>
@@ -838,5 +838,5 @@
         <origin xyz="-8.73189226654e-10 1.36059566391e-13 0.05" rpy="-3.35384399272e-13 -3.58979304269e-09 1.3471843864e-14" />
         <geometry>
-          <mesh filename="package://cleany_description/meshes/Lower_Arm_Motor.stl" scale="1 1 1" />
+          <mesh filename="package://cleany_description/meshes/${arm_collision_directory}Lower_Arm_Motor.stl" scale="1 1 1" />
         </geometry>
       </collision>
@@ -869,5 +869,5 @@
         <origin xyz="-1.35745237707e-09 1.73749903354e-14 1.81328422329e-13" rpy="1.62630325873e-17 5.48606299278e-17 -3.58979312942e-09" />
         <geometry>
-          <mesh filename="package://cleany_description/meshes/Wrist_Pitch_Roll.stl" scale="1 1 1" />
+          <mesh filename="package://cleany_description/meshes/${arm_collision_directory}Wrist_Pitch_Roll.stl" scale="1 1 1" />
         </geometry>
       </collision>
@@ -1005,9 +1005,9 @@
         <collision name="head_mast_cad_collision">
           <origin xyz="-0.440000013266 -0.00499883242047 -0.6" rpy="-1.73472347598e-18 6.93889390391e-18 -2.65358979331e-06" />
-          <geometry><mesh filename="package://cleany_description/meshes/cad_frame/topbase1.stl" scale="1 1 1" /></geometry>
+          <geometry><mesh filename="package://cleany_description/meshes/${arm_collision_directory}cad_frame/topbase1.stl" scale="1 1 1" /></geometry>
         </collision>
         <collision name="lower_head_mount_cad_collision">
           <origin xyz="-0.297999984077 0.00600079076974 -0.6875" rpy="-5.90619133461e-17 6.93889390391e-18 3.13999734641" />
-          <geometry><mesh filename="package://cleany_description/meshes/topbase2.stl" scale="0.001 0.001 0.001" /></geometry>
+          <geometry><mesh filename="package://cleany_description/meshes/${arm_collision_directory}topbase2.stl" scale="0.001 0.001 0.001" /></geometry>
         </collision>
       </xacro:if>
@@ -1056,9 +1056,9 @@
         <collision name="head_pan_bracket_cad_collision">
           <origin xyz="-0.335000013266 -0.00499883772765 -0.923" rpy="8.67361737988e-19 -5.55111512313e-17 -2.65358979336e-06" />
-          <geometry><mesh filename="package://cleany_description/meshes/tophead1.stl" scale="0.001 0.001 0.001" /></geometry>
+          <geometry><mesh filename="package://cleany_description/meshes/${arm_collision_directory}tophead1.stl" scale="0.001 0.001 0.001" /></geometry>
         </collision>
         <collision name="head_pan_motor_cad_collision">
           <origin xyz="1.16999997611 -0.00900283138028 0.262" rpy="-3.14159201945 -1.57000000101 3.14159063414" />
-          <geometry><mesh filename="package://cleany_description/meshes/tophead4.stl" scale="0.001 0.001 0.001" /></geometry>
+          <geometry><mesh filename="package://cleany_description/meshes/${arm_collision_directory}tophead4.stl" scale="0.001 0.001 0.001" /></geometry>
         </collision>
       </xacro:if>
@@ -1099,9 +1099,9 @@
         <collision name="head_tilt_bracket_cad_collision">
           <origin xyz="0.162649962825 -0.00600113446269 -1.16815" rpy="-6.20163642662e-17 4.55026099265e-18 -5.31076937972e-06" />
-          <geometry><mesh filename="package://cleany_description/meshes/tophead5.stl" scale="0.001 0.001 0.001" /></geometry>
+          <geometry><mesh filename="package://cleany_description/meshes/${arm_collision_directory}tophead5.stl" scale="0.001 0.001 0.001" /></geometry>
         </collision>
         <collision name="head_tilt_motor_cad_collision">
           <origin xyz="0.162649962825 -0.00600113446269 -1.16815" rpy="-3.56491214576e-17 -1.75849280414e-18 -5.31076937974e-06" />
-          <geometry><mesh filename="package://cleany_description/meshes/tophead6.stl" scale="0.001 0.001 0.001" /></geometry>
+          <geometry><mesh filename="package://cleany_description/meshes/${arm_collision_directory}tophead6.stl" scale="0.001 0.001 0.001" /></geometry>
         </collision>
       </xacro:if>
