Commit message: feat(manipulation): add physical grasp planning and execution foundation

File: ros2_ws/src/cleany_moveit_config/config/cleany_mock.urdf.xacro (robot description, xacro)
@@ -1,13 +1,19 @@
 <?xml version="1.0"?>
 <robot name="cleany" xmlns:xacro="http://www.ros.org/wiki/xacro">
+  <xacro:arg name="include_head_camera" default="false"/>
+  <xacro:arg name="head_tilt_initial" default="0.405"/>
   <!-- Reuse the canonical geometry; this file only adds a mock ros2_control system. -->
   <xacro:include filename="$(find cleany_description)/urdf/materials.xacro"/>
   <xacro:include filename="$(find cleany_description)/urdf/cleany_geometry.xacro"/>
+  <xacro:include filename="$(find cleany_description)/urdf/head_camera.xacro"/>
   <xacro:cleany_robot_geometry/>
-  <xacro:macro name="cleany_mock_joint" params="joint_name">
+  <xacro:if value="$(arg include_head_camera)">
+    <xacro:cleany_head_camera/>
+  </xacro:if>
+  <xacro:macro name="cleany_mock_joint" params="joint_name initial_value:=0.0">
     <joint name="${joint_name}">
       <command_interface name="position"/>
       <state_interface name="position">
-        <param name="initial_value">0.0</param>
+        <param name="initial_value">${initial_value}</param>
       </state_interface>
       <state_interface name="velocity"/>
@@ -30,4 +36,8 @@
     <xacro:cleany_mock_joint joint_name="right_wrist_roll_joint"/>
     <xacro:cleany_mock_joint joint_name="right_gripper_joint"/>
+    <xacro:if value="$(arg include_head_camera)">
+      <xacro:cleany_mock_joint joint_name="head_pan_joint" initial_value="0.023"/>
+      <xacro:cleany_mock_joint joint_name="head_tilt_joint" initial_value="$(arg head_tilt_initial)"/>
+    </xacro:if>
   </ros2_control>
 </robot>
